File: SATA.kicad_sch (KiCad schematic)
At the start: 30 parts, among them J1 Bus_M.2_Socket_B, U12 JMS578, U13 CAT250xxx, U2 ASEK-32.768KHZ-L-R-T, Y4 30Mhz

Commit message: change cad data
Parts:
- added C12, C14, C17: 0.1uF, Capacitor_SMD:C_0402_1005Metric_Pad0.74x0.62mm_HandSolder, symbol Device:C
- added C13: 0.01uF, Capacitor_SMD:C_0402_1005Metric_Pad0.74x0.62mm_HandSolder, symbol Device:C
- renumbered C76 to C100, C77 to C103, C78 to C104, C2 to C11, C46 to C68, C47 to C69, C48 to C70, C49 to C71, C50 to C72, C53 to C75, C54 to C76, C55 to C77, C56 to C78, C57 to C79, C58 to C80, C63 to C81, C66 to C89, C65 to C90, C67 to C91, C74 to C98, D7 to D8, J1 to J3, R40 to R49, R43 to R58, R45 to R60, U12 to U13, U13 to U14, U2 to U4, Y4 to Y5
Connections:
- net SATA_RXN: now also C13.2; no longer J3.43 (PERp0/SATA-B-)
- net SATA_RXP: now also C12.2; no longer J3.41 (PERn0/SATA-B+)
- net SATA_TXN: now also C14.2; no longer J3.47 (PETn0/SATA-A-)
- net SATA_TXP: now also C17.2; no longer J3.49 (PETp0/SATA-A+)
- new net: C13.1, J3.43 (PERp0/SATA-B-)
- new net: C14.1, J3.47 (PETn0/SATA-A-)
- new net: C17.1, J3.49 (PETp0/SATA-A+)
- new net: C12.1, J3.41 (PERn0/SATA-B+)
- no-connect marks 9 -> 11
Other:
- moved on the sheet: C11, C71, J3, U4

Commit message: change clearance
Changed lines of the file:
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@@
 	(wire
 		(pts
-			(xy 180.34 46.99) (xy 180.34 49.53)
-		)
-		(stroke
-			(width 0)
-			(type default)
-		)
-	)
-	(wire
-		(pts
 			(xy 107.95 137.16) (xy 107.95 128.27)
 		)
@@
 	(wire
 		(pts
-			(xy 175.26 59.69) (xy 180.34 59.69)
+			(xy 175.26 57.15) (xy 180.34 57.15)
 		)
 		(stroke
@@
 	(wire
 		(pts
-			(xy 180.34 49.53) (xy 175.26 49.53)
+			(xy 180.34 46.99) (xy 175.26 46.99)
 		)
 		(stroke
@@
 	(wire
 		(pts
-			(xy 180.34 57.15) (xy 180.34 59.69)
-		)
-		(stroke
-			(width 0)
-			(type default)
-		)
-	)
-	(wire
-		(pts
 			(xy 134.62 175.26) (xy 146.05 175.26)
 		)
@@
 	)
 	(label "SATA_RXN"
-		(at 175.26 59.69 180)
+		(at 175.26 57.15 180)
 		(fields_autoplaced yes)
 		(effects
@@
 	)
 	(label "SATA_TXP"
-		(at 175.26 49.53 180)
+		(at 175.26 46.99 180)
 		(fields_autoplaced yes)
 		(effects
@@
 		(dnp no)
 		(property "Reference" "C13"
-			(at 178.054 55.372 90)
+			(at 188.722 55.372 90)
 			(effects
 				(font
@@
 		)
 		(property "Value" "0.01uF"
-			(at 178.054 57.912 90)
+			(at 188.722 57.912 90)
 			(effects
 				(font
@@
 		(dnp no)
 		(property "Reference" "C17"
-			(at 179.578 41.91 90)
+			(at 189.484 45.72 90)
 			(effects
 				(font
@@
 		)
 		(property "Value" "0.1uF"
-			(at 179.578 44.45 90)
+			(at 189.484 48.26 90)
 			(effects
 				(font
@@
 		(dnp no)
 		(property "Reference" "C12"
-			(at 179.324 64.77 90)
+			(at 188.976 60.706 90)
 			(effects
 				(font
@@
 		)
 		(property "Value" "0.1uF"
-			(at 179.324 67.31 90)
+			(at 188.976 63.246 90)
 			(effects
 				(font

Commit message: remove efuse
Parts:
- renumbered C14 to C11, C17 to C13, C68 to C58, C69 to C59, C70 to C60, C71 to C61, C72 to C62, C75 to C65, C76 to C66, C77 to C67, C78 to C68, C79 to C69, C11 to C7, C80 to C70, C81 to C71, C90 to C79, C12 to C8, C89 to C80, C91 to C81, C98 to C82, C13 to C9, C100 to C91, C103 to C92, C104 to C94, R49 to R48, R58 to R57, R60 to R58, U13 to U14, U14 to U15, Y5 to Y4
Changed lines of the file:
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@@
 		(dnp no)
 		(fields_autoplaced yes)
-		(property "Reference" "C71"
+		(property "Reference" "C61"
 			(at 152.4 118.1099 0)
 			(effects
@@
 			(project "mainboard4"
 				(path "/dd07ab80-a59c-44f4-ac7d-849e21e1384e/5db2a135-33ff-4812-ab9d-2394338dfef8"
-					(reference "C71")
+					(reference "C61")
 					(unit 1)
 				)
@@
 		(on_board yes)
 		(dnp no)
-		(property "Reference" "C91"
+		(property "Reference" "C81"
 			(at 88.9 177.8 0)
 			(effects
@@
 			(project "mainboard4"
 				(path "/dd07ab80-a59c-44f4-ac7d-849e21e1384e/5db2a135-33ff-4812-ab9d-2394338dfef8"
-					(reference "C91")
+					(reference "C81")
 					(unit 1)
 				)
@@
 		(dnp no)
 		(fields_autoplaced yes)
-		(property "Reference" "C100"
+		(property "Reference" "C91"
 			(at 39.37 177.7999 0)
 			(effects
@@
 			(project "mainboard4"
 				(path "/dd07ab80-a59c-44f4-ac7d-849e21e1384e/5db2a135-33ff-4812-ab9d-2394338dfef8"
-					(reference "C100")
+					(reference "C91")
 					(unit 1)
 				)
@@
 		(dnp no)
 		(fields_autoplaced yes)
-		(property "Reference" "C75"
+		(property "Reference" "C65"
 			(at 139.7 130.8099 0)
 			(effects
@@
 			(project "mainboard4"
 				(path "/dd07ab80-a59c-44f4-ac7d-849e21e1384e/5db2a135-33ff-4812-ab9d-2394338dfef8"
-					(reference "C75")
+					(reference "C65")
 					(unit 1)
 				)
@@
 		(dnp no)
 		(fields_autoplaced yes)
-		(property "Reference" "C77"
+		(property "Reference" "C67"
 			(at 125.73 177.7999 0)
 			(effects
@@
 			(project "mainboard4"
 				(path "/dd07ab80-a59c-44f4-ac7d-849e21e1384e/5db2a135-33ff-4812-ab9d-2394338dfef8"
-					(reference "C77")
+					(reference "C67")
 					(unit 1)
 				)
@@
 		(dnp no)
 		(fields_autoplaced yes)
-		(property "Reference" "C89"
+		(property "Reference" "C80"
 			(at 62.23 177.7999 0)
 			(effects
@@
 			(project "mainboard4"
 				(path "/dd07ab80-a59c-44f4-ac7d-849e21e1384e/5db2a135-33ff-4812-ab9d-2394338dfef8"
-					(reference "C89")
+					(reference "C80")
 					(unit 1)
 				)
@@
 		(dnp no)
 		(fields_autoplaced yes)
-		(property "Reference" "C78"
+		(property "Reference" "C68"
 			(at 149.86 177.7999 0)
 			(effects
@@
 			(project "mainboard4"
 				(path "/dd07ab80-a59c-44f4-ac7d-849e21e1384e/5db2a135-33ff-4812-ab9d-2394338dfef8"
-					(reference "C78")
+					(reference "C68")
 					(unit 1)
 				)
@@
 		(on_board yes)
 		(dnp no)
-		(property "Reference" "C13"
+		(property "Reference" "C9"
 			(at 188.722 55.372 90)
 			(effects
@@
 			(project "mainboard4"
 				(path "/dd07ab80-a59c-44f4-ac7d-849e21e1384e/5db2a135-33ff-4812-ab9d-2394338dfef8"
-					(reference "C13")
+					(reference "C9")
 					(unit 1)
 				)
@@
 		(dnp no)
 		(fields_autoplaced yes)
-		(property "Reference" "C103"
+		(property "Reference" "C92"
 			(at 53.34 109.2199 0)
 			(effects
@@
 			(project ""
 				(path "/dd07ab80-a59c-44f4-ac7d-849e21e1384e/5db2a135-33ff-4812-ab9d-2394338dfef8"
-					(reference "C103")
+					(reference "C92")
 					(unit 1)
 				)
@@
 		(dnp no)
 		(fields_autoplaced yes)
-		(property "Reference" "Y5"
+		(property "Reference" "Y4"
 			(at 152.4 60.9914 0)
 			(effects
@@
 			(project "mainboard4"
 				(path "/dd07ab80-a59c-44f4-ac7d-849e21e1384e/5db2a135-33ff-4812-ab9d-2394338dfef8"
-					(reference "Y5")
+					(reference "Y4")
 					(unit 1)
 				)
@@
 		(dnp no)
 		(fields_autoplaced yes)
-		(property "Reference" "C90"
+		(property "Reference" "C79"
 			(at 64.77 92.7099 0)
 			(effects
@@
 			(project "mainboard4"
 				(path "/dd07ab80-a59c-44f4-ac7d-849e21e1384e/5db2a135-33ff-4812-ab9d-2394338dfef8"
-					(reference "C90")
+					(reference "C79")
 					(unit 1)
 				)
@@
 		(dnp no)
 		(fields_autoplaced yes)
-		(property "Reference" "C68"
+		(property "Reference" "C58"
 			(at 138.43 177.7999 0)
 			(effects
@@
 			(project "mainboard4"
 				(path "/dd07ab80-a59c-44f4-ac7d-849e21e1384e/5db2a135-33ff-4812-ab9d-2394338dfef8"
-					(reference "C68")
+					(reference "C58")
 					(unit 1)
 				)
@@
 		(dnp no)
 		(fields_autoplaced yes)
-		(property "Reference" "C70"
+		(property "Reference" "C60"
 			(at 77.47 177.7999 0)
 			(effects
@@
 			(project "mainboard4"
 				(path "/dd07ab80-a59c-44f4-ac7d-849e21e1384e/5db2a135-33ff-4812-ab9d-2394338dfef8"
-					(reference "C70")
+					(reference "C60")
 					(unit 1)
 				)
@@
 		(dnp no)
 		(fields_autoplaced yes)
-		(property "Reference" "C98"
+		(property "Reference" "C82"
 			(at 50.8 177.7999 0)
 			(effects
@@
 			(project "mainboard4"
 				(path "/dd07ab80-a59c-44f4-ac7d-849e21e1384e/5db2a135-33ff-4812-ab9d-2394338dfef8"
-					(reference "C98")
+					(reference "C82")
 					(unit 1)
 				)
@@
 		(on_board yes)
 		(dnp no)
-		(property "Reference" "C72"
+		(property "Reference" "C62"
 			(at 126.746 69.596 0)
 			(effects
@@
 			(project "mainboard4"
 				(path "/dd07ab80-a59c-44f4-ac7d-849e21e1384e/5db2a135-33ff-4812-ab9d-2394338dfef8"
-					(reference "C72")
+					(reference "C62")
 					(unit 1)
 				)
@@
 		(on_board yes)
 		(dnp no)
-		(property "Reference" "C69"
+		(property "Reference" "C59"
 			(at 161.29 177.7999 0)
 			(effects
@@
 			(project "mainboard4"
 				(path "/dd07ab80-a59c-44f4-ac7d-849e21e1384e/5db2a135-33ff-4812-ab9d-2394338dfef8"
-					(reference "C69")
+					(reference "C59")
 					(unit 1)
 				)
@@
 		(on_board yes)
 		(dnp no)
-		(property "Reference" "C11"
+		(property "Reference" "C7"
 			(at 246.761 152.5016 0)
 			(effects
@@
 			(project "mainboard4"
 				(path "/dd07ab80-a59c-44f4-ac7d-849e21e1384e/5db2a135-33ff-4812-ab9d-2394338dfef8"
-					(reference "C11")
+					(reference "C7")
 					(unit 1)
 				)
@@
 		(on_board yes)
 		(dnp no)
-		(property "Reference" "C14"
+		(property "Reference" "C11"
 			(at 188.976 50.546 90)
 			(effects
@@
 			(project "mainboard4"
 				(path "/dd07ab80-a59c-44f4-ac7d-849e21e1384e/5db2a135-33ff-4812-ab9d-2394338dfef8"
-					(reference "C14")
+					(reference "C11")
 					(unit 1)
 				)
@@
 		(dnp no)
 		(fields_autoplaced yes)
-		(property "Reference" "R49"
+		(property "Reference" "R48"
 			(at 39.37 142.24 90)
 			(effects
@@
 			(project "mainboard4"
 				(path "/dd07ab80-a59c-44f4-ac7d-849e21e1384e/5db2a135-33ff-4812-ab9d-2394338dfef8"
-					(reference "R49")
+					(reference "R48")
 					(unit 1)
 				)
@@
 		(dnp no)
 		(fields_autoplaced yes)
-		(property "Reference" "R58"
+		(property "Reference" "R57"
 			(at 85.09 68.58 90)
 			(effects
@@
 			(project ""
 				(path "/dd07ab80-a59c-44f4-ac7d-849e21e1384e/5db2a135-33ff-4812-ab9d-2394338dfef8"
-					(reference "R58")
+					(reference "R57")
 					(unit 1)
 				)
@@
 		(dnp no)
 		(fields_autoplaced yes)
-		(property "Reference" "C80"
+		(property "Reference" "C70"
 			(at 102.87 177.7999 0)
 			(effects
@@
 			(project "mainboard4"
 				(path "/dd07ab80-a59c-44f4-ac7d-849e21e1384e/5db2a135-33ff-4812-ab9d-2394338dfef8"
-					(reference "C80")
+					(reference "C70")
 					(unit 1)
 				)
@@
 		(on_board yes)
 		(dnp no)
-		(property "Reference" "U13"
+		(property "Reference" "U14"
 			(at 106.426 58.674 0)
 			(effects
@@
 			(project ""
 				(path "/dd07ab80-a59c-44f4-ac7d-849e21e1384e/5db2a135-33ff-4812-ab9d-2394338dfef8"
-					(reference "U13")
+					(reference "U14")
 					(unit 1)
 				)
@@
 		(dnp no)
 		(fields_autoplaced yes)
-		(property "Reference" "U14"
+		(property "Reference" "U15"
 			(at 107.6041 146.05 0)
 			(effects
@@
 			(project ""
 				(path "/dd07ab80-a59c-44f4-ac7d-849e21e1384e/5db2a135-33ff-4812-ab9d-2394338dfef8"
-					(reference "U14")
+					(reference "U15")
 					(unit 1)
 				)
@@
 		(on_board yes)
 		(dnp no)
-		(property "Reference" "C79"
+		(property "Reference" "C69"
 			(at 25.4 177.8 0)
 			(effects
@@
 			(project "mainboard4"
 				(path "/dd07ab80-a59c-44f4-ac7d-849e21e1384e/5db2a135-33ff-4812-ab9d-2394338dfef8"
-					(reference "C79")
+					(reference "C69")
 					(unit 1)
 				)
@@
 		(on_board yes)
 		(dnp no)
-		(property "Reference" "C76"
+		(property "Reference" "C66"
 			(at 150.368 70.358 0)
 			(effects
@@
 			(project "mainboard4"
 				(path "/dd07ab80-a59c-44f4-ac7d-849e21e1384e/5db2a135-33ff-4812-ab9d-2394338dfef8"
-					(reference "C76")
+					(reference "C66")
 					(unit 1)
 				)
@@
 		(on_board yes)
 		(dnp no)
-		(property "Reference" "C17"
+		(property "Reference" "C13"
 			(at 189.484 45.72 90)
 			(effects
@@
 			(project "mainboard4"
 				(path "/dd07ab80-a59c-44f4-ac7d-849e21e1384e/5db2a135-33ff-4812-ab9d-2394338dfef8"
-					(reference "C17")
+					(reference "C13")
 					(unit 1)
 				)
@@
 		(on_board yes)
 		(dnp no)
-		(property "Reference" "C104"
+		(property "Reference" "C94"
 			(at 59.69 114.808 0)
 			(effects
@@
 			(project "mainboard4"
 				(path "/dd07ab80-a59c-44f4-ac7d-849e21e1384e/5db2a135-33ff-4812-ab9d-2394338dfef8"
-					(reference "C104")
+					(reference "C94")
 					(unit 1)
 				)
@@
 		(on_board yes)
 		(dnp no)
-		(property "Reference" "C12"
+		(property "Reference" "C8"
 			(at 188.976 60.706 90)
 			(effects
@@
 			(project "mainboard4"
 				(path "/dd07ab80-a59c-44f4-ac7d-849e21e1384e/5db2a135-33ff-4812-ab9d-2394338dfef8"
-					(reference "C12")
+					(reference "C8")
 					(unit 1)
 				)
@@
 		(dnp no)
 		(fields_autoplaced yes)
-		(property "Reference" "C81"
+		(property "Reference" "C71"
 			(at 114.3 177.7999 0)
 			(effects
@@
 			(project "mainboard4"
 				(path "/dd07ab80-a59c-44f4-ac7d-849e21e1384e/5db2a135-33ff-4812-ab9d-2394338dfef8"
-					(reference "C81")
+					(reference "C71")
 					(unit 1)
 				)
@@
 		(dnp no)
 		(fields_autoplaced yes)
-		(property "Reference" "R60"
+		(property "Reference" "R58"
 			(at 63.5 85.0899 0)
 			(effects
@@
 			(project "mainboard4"
 				(path "/dd07ab80-a59c-44f4-ac7d-849e21e1384e/5db2a135-33ff-4812-ab9d-2394338dfef8"
-					(reference "R60")
+					(reference "R58")
 					(unit 1)
 				)

Commit message: change sata sch
Parts:
- added C136, C137, C139: 0.1uF, Capacitor_SMD:C_0402_1005Metric_Pad0.74x0.62mm_HandSolder, symbol Device:C
- added C138: 0.01uF, Capacitor_SMD:C_0402_1005Metric_Pad0.74x0.62mm_HandSolder, symbol Device:C
Connections:
- net +3.3V: now also C136.1, C137.1, C138.1, C139.1
- net GND: now also C136.2, C137.2, C138.2, C139.2

Commit message: add sata capacitor
Parts:
- C1: renamed from C137; footprint Capacitor_SMD:C_0402_1005Metric_Pad0.74x0.62mm_HandSolder -> Capacitor_SMD:C_0603_1608Metric
- C10: renamed from C138; footprint Capacitor_SMD:C_0402_1005Metric_Pad0.74x0.62mm_HandSolder -> Capacitor_SMD:C_0603_1608Metric
- C2: renamed from C136; footprint Capacitor_SMD:C_0402_1005Metric_Pad0.74x0.62mm_HandSolder -> Capacitor_SMD:C_0603_1608Metric
- C9: renamed from C139; footprint Capacitor_SMD:C_0402_1005Metric_Pad0.74x0.62mm_HandSolder -> Capacitor_SMD:C_0603_1608Metric
- renumbered C91 to C101, C92 to C102, C94 to C103, C7 to C11, C8 to C12, C9 to C13, C11 to C15, C13 to C17, C60 to C68, C59 to C69, C58 to C70, C61 to C71, C62 to C72, C65 to C75, C66 to C76, C67 to C77, C68 to C78, C69 to C79, C70 to C80, C71 to C81, C81 to C89, C80 to C90, C79 to C91, C82 to C92, D8 to D11, R48 to R49, R57 to R54, R58 to R60

Commit message: change design
Parts:
- renumbered C102 to C103, C76 to C75, C75 to C76, C92 to C89, C89 to C90, C90 to C91, C91 to C92, C103 to C93
Changed lines of the file:
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@@
 		(on_board yes)
 		(dnp no)
-		(property "Reference" "C89"
+		(property "Reference" "C90"
 			(at 88.9 177.8 0)
 			(effects
@@
 			(project "mainboard4"
 				(path "/dd07ab80-a59c-44f4-ac7d-849e21e1384e/5db2a135-33ff-4812-ab9d-2394338dfef8"
-					(reference "C89")
+					(reference "C90")
 					(unit 1)
 				)
@@
 		(dnp no)
 		(fields_autoplaced yes)
-		(property "Reference" "C75"
+		(property "Reference" "C76"
 			(at 139.7 130.8099 0)
 			(effects
@@
 			(project "mainboard4"
 				(path "/dd07ab80-a59c-44f4-ac7d-849e21e1384e/5db2a135-33ff-4812-ab9d-2394338dfef8"
-					(reference "C75")
+					(reference "C76")
 					(unit 1)
 				)
@@
 		(dnp no)
 		(fields_autoplaced yes)
-		(property "Reference" "C90"
+		(property "Reference" "C91"
 			(at 62.23 177.7999 0)
 			(effects
@@
 			(project "mainboard4"
 				(path "/dd07ab80-a59c-44f4-ac7d-849e21e1384e/5db2a135-33ff-4812-ab9d-2394338dfef8"
-					(reference "C90")
+					(reference "C91")
 					(unit 1)
 				)
@@
 		(dnp no)
 		(fields_autoplaced yes)
-		(property "Reference" "C102"
+		(property "Reference" "C103"
 			(at 53.34 109.2199 0)
 			(effects
@@
 			(project ""
 				(path "/dd07ab80-a59c-44f4-ac7d-849e21e1384e/5db2a135-33ff-4812-ab9d-2394338dfef8"
-					(reference "C102")
+					(reference "C103")
 					(unit 1)
 				)
@@
 		(dnp no)
 		(fields_autoplaced yes)
-		(property "Reference" "C91"
+		(property "Reference" "C92"
 			(at 64.77 92.7099 0)
 			(effects
@@
 			(project "mainboard4"
 				(path "/dd07ab80-a59c-44f4-ac7d-849e21e1384e/5db2a135-33ff-4812-ab9d-2394338dfef8"
-					(reference "C91")
+					(reference "C92")
 					(unit 1)
 				)
@@
 		(dnp no)
 		(fields_autoplaced yes)
-		(property "Reference" "C92"
+		(property "Reference" "C89"
 			(at 50.8 177.7999 0)
 			(effects
@@
 			(project "mainboard4"
 				(path "/dd07ab80-a59c-44f4-ac7d-849e21e1384e/5db2a135-33ff-4812-ab9d-2394338dfef8"
-					(reference "C92")
+					(reference "C89")
 					(unit 1)
 				)
@@
 		(on_board yes)
 		(dnp no)
-		(property "Reference" "C76"
+		(property "Reference" "C75"
 			(at 150.368 70.358 0)
 			(effects
@@
 			(project "mainboard4"
 				(path "/dd07ab80-a59c-44f4-ac7d-849e21e1384e/5db2a135-33ff-4812-ab9d-2394338dfef8"
-					(reference "C76")
+					(reference "C75")
 					(unit 1)
 				)
@@
 		(on_board yes)
 		(dnp no)
-		(property "Reference" "C103"
+		(property "Reference" "C93"
 			(at 59.69 114.808 0)
 			(effects
@@
 			(project "mainboard4"
 				(path "/dd07ab80-a59c-44f4-ac7d-849e21e1384e/5db2a135-33ff-4812-ab9d-2394338dfef8"
-					(reference "C103")
+					(reference "C93")
 					(unit 1)
 				)

Commit message: add logp
Parts:
- renumbered C92 to C90, C90 to C91, C91 to C92, R49 to R46, R54 to R51, R60 to R58
Changed lines of the file:
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@@
 	(label "CS"
 		(at 107.95 137.16 90)
-		(fields_autoplaced yes)
 		(effects
 			(font
@@
 	(label "SATA_RXP"
 		(at 175.26 62.23 180)
-		(fields_autoplaced yes)
 		(effects
 			(font
@@
 	(label "SATA_RXP"
 		(at 110.49 66.04 180)
-		(fields_autoplaced yes)
 		(effects
 			(font
@@
 	(label "SCLK"
 		(at 120.65 153.67 180)
-		(fields_autoplaced yes)
 		(effects
 			(font
@@
 	(label "AV3V3"
 		(at 15.24 175.26 0)
-		(fields_autoplaced yes)
 		(effects
 			(font
@@
 	(label "SATA_RXN"
 		(at 107.95 68.58 180)
-		(fields_autoplaced yes)
 		(effects
 			(font
@@
 	(label "AV1V2"
 		(at 148.59 97.79 180)
-		(fields_autoplaced yes)
 		(effects
 			(font
@@
 	(label "AV3V3"
 		(at 87.63 153.67 0)
-		(fields_autoplaced yes)
 		(effects
 			(font
@@
 	(label "SI"
 		(at 119.38 156.21 180)
-		(fields_autoplaced yes)
 		(effects
 			(font
@@
 	(label "SI"
 		(at 105.41 137.16 90)
-		(fields_autoplaced yes)
 		(effects
 			(font
@@
 	(label "SATA_TXN"
 		(at 102.87 71.12 180)
-		(fields_autoplaced yes)
 		(effects
 			(font
@@
 	(label "AV3V3"
 		(at 73.66 110.49 0)
-		(fields_autoplaced yes)
 		(effects
 			(font
@@
 	(label "SCLK"
 		(at 100.33 137.16 90)
-		(fields_autoplaced yes)
 		(effects
 			(font
@@
 	(label "SATA_TXN"
 		(at 175.26 52.07 180)
-		(fields_autoplaced yes)
 		(effects
 			(font
@@
 	(label "AV1V2"
 		(at 73.66 175.26 180)
-		(fields_autoplaced yes)
 		(effects
 			(font
@@
 	(label "AV1V2"
 		(at 148.59 90.17 180)
-		(fields_autoplaced yes)
 		(effects
 			(font
@@
 	(label "HDD_LED"
 		(at 113.03 137.16 90)
-		(fields_autoplaced yes)
 		(effects
 			(font
@@
 	(label "AV3V3"
 		(at 60.96 73.66 270)
-		(fields_autoplaced yes)
 		(effects
 			(font
@@
 	(label "AV3V3"
 		(at 77.47 92.71 0)
-		(fields_autoplaced yes)
 		(effects
 			(font
@@
 	(label "AV1V2"
 		(at 113.03 71.12 270)
-		(fields_autoplaced yes)
 		(effects
 			(font
@@
 	(label "AV3V3"
 		(at 110.49 137.16 90)
-		(fields_autoplaced yes)
 		(effects
 			(font
@@
 	(label "SATA_RXN"
 		(at 175.26 57.15 180)
-		(fields_autoplaced yes)
 		(effects
 			(font
@@
 	(label "HDD_LED"
 		(at 31.75 148.59 180)
-		(fields_autoplaced yes)
 		(effects
 			(font
@@
 	(label "AV1V2"
 		(at 77.47 95.25 0)
-		(fields_autoplaced yes)
 		(effects
 			(font
@@
 	(label "SO"
 		(at 119.38 158.75 180)
-		(fields_autoplaced yes)
 		(effects
 			(font
@@
 	(label "AV3V3"
 		(at 87.63 156.21 0)
-		(fields_autoplaced yes)
 		(effects
 			(font
@@
 	(label "AV1V2"
 		(at 105.41 71.12 270)
-		(fields_autoplaced yes)
 		(effects
 			(font
@@
 	(label "SATA_TXP"
 		(at 175.26 46.99 180)
-		(fields_autoplaced yes)
 		(effects
 			(font
@@
 	(label "SATA_TXP"
 		(at 100.33 73.66 180)
-		(fields_autoplaced yes)
 		(effects
 			(font
@@
 	(label "AV3V3"
 		(at 158.75 115.57 180)
-		(fields_autoplaced yes)
 		(effects
 			(font
@@
 	(label "AV1V2"
 		(at 102.87 137.16 90)
-		(fields_autoplaced yes)
 		(effects
 			(font
@@
 	(label "AV3V3"
 		(at 105.41 148.59 180)
-		(fields_autoplaced yes)
 		(effects
 			(font
@@
 	(label "AV1V2"
 		(at 49.53 105.41 180)
-		(fields_autoplaced yes)
 		(effects
 			(font
@@
 	(label "SO"
 		(at 97.79 137.16 90)
-		(fields_autoplaced yes)
 		(effects
 			(font
@@
 	(label "AV1V2"
 		(at 148.59 105.41 180)
-		(fields_autoplaced yes)
 		(effects
 			(font
@@
 	(label "CS"
 		(at 91.44 158.75 0)
-		(fields_autoplaced yes)
 		(effects
 			(font
@@
 	(label "AV1V2"
 		(at 118.11 137.16 90)
-		(fields_autoplaced yes)
 		(effects
 			(font
@@
 		(shape output)
 		(at 132.08 92.71 0)
-		(fields_autoplaced yes)
 		(effects
 			(font
@@
 		(shape bidirectional)
 		(at 132.08 113.03 0)
-		(fields_autoplaced yes)
 		(effects
 			(font
@@
 		(shape output)
 		(at 132.08 95.25 0)
-		(fields_autoplaced yes)
 		(effects
 			(font
@@
 		(shape input)
 		(at 132.08 100.33 0)
-		(fields_autoplaced yes)
 		(effects
 			(font
@@
 		(shape bidirectional)
 		(at 132.08 118.11 0)
-		(fields_autoplaced yes)
 		(effects
 			(font
@@
 		(shape input)
 		(at 132.08 102.87 0)
-		(fields_autoplaced yes)
 		(effects
 			(font
@@
 		(on_board yes)
 		(dnp no)
-		(property "Reference" "C90"
+		(property "Reference" "C91"
 			(at 88.9 177.8 0)
 			(effects
@@
 			(project "mainboard4"
 				(path "/dd07ab80-a59c-44f4-ac7d-849e21e1384e/5db2a135-33ff-4812-ab9d-2394338dfef8"
-					(reference "C90")
+					(reference "C91")
 					(unit 1)
 				)
@@
 		(dnp no)
 		(fields_autoplaced yes)
-		(property "Reference" "C91"
+		(property "Reference" "C92"
 			(at 62.23 177.7999 0)
 			(effects
@@
 			(project "mainboard4"
 				(path "/dd07ab80-a59c-44f4-ac7d-849e21e1384e/5db2a135-33ff-4812-ab9d-2394338dfef8"
-					(reference "C91")
+					(reference "C92")
 					(unit 1)
 				)
@@
 		(dnp no)
 		(fields_autoplaced yes)
-		(property "Reference" "C92"
+		(property "Reference" "C90"
 			(at 64.77 92.7099 0)
 			(effects
@@
 			(project "mainboard4"
 				(path "/dd07ab80-a59c-44f4-ac7d-849e21e1384e/5db2a135-33ff-4812-ab9d-2394338dfef8"
-					(reference "C92")
+					(reference "C90")
 					(unit 1)
 				)
@@
 		(dnp no)
 		(fields_autoplaced yes)
-		(property "Reference" "R49"
+		(property "Reference" "R46"
 			(at 39.37 142.24 90)
 			(effects
@@
 			(project "mainboard4"
 				(path "/dd07ab80-a59c-44f4-ac7d-849e21e1384e/5db2a135-33ff-4812-ab9d-2394338dfef8"
-					(reference "R49")
+					(reference "R46")
 					(unit 1)
 				)
@@
 		(dnp no)
 		(fields_autoplaced yes)
-		(property "Reference" "R54"
+		(property "Reference" "R51"
 			(at 85.09 68.58 90)
 			(effects
@@
 			(project ""
 				(path "/dd07ab80-a59c-44f4-ac7d-849e21e1384e/5db2a135-33ff-4812-ab9d-2394338dfef8"
-					(reference "R54")
+					(reference "R51")
 					(unit 1)
 				)
@@
 		(dnp no)
 		(fields_autoplaced yes)
-		(property "Reference" "R60"
+		(property "Reference" "R58"
 			(at 63.5 85.0899 0)
 			(effects
@@
 			(project "mainboard4"
 				(path "/dd07ab80-a59c-44f4-ac7d-849e21e1384e/5db2a135-33ff-4812-ab9d-2394338dfef8"
-					(reference "R60")
+					(reference "R58")
 					(unit 1)
 				)
