File: SATA.kicad_sch (KiCad schematic)
At the start: 38 parts, among them J3 Bus_M.2_Socket_B, U14 JMS578, U15 CAT250xxx, U4 ASEK-32.768KHZ-L-R-T, Y4 30Mhz

Commit message: add usb
Connections:
- net +5V renamed VBUS
Changed lines of the file:
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@@
 	)
 	(junction
-		(at 135.89 128.27)
-		(diameter 0)
-		(color 0 0 0 0)
-	)
-	(junction
 		(at 80.01 128.27)
 		(diameter 0)
@@
 	(label "CS"
 		(at 107.95 137.16 90)
+		(fields_autoplaced yes)
 		(effects
 			(font
@@
 	(label "SATA_RXP"
 		(at 175.26 62.23 180)
+		(fields_autoplaced yes)
 		(effects
 			(font
@@
 	(label "SATA_RXP"
 		(at 110.49 66.04 180)
+		(fields_autoplaced yes)
 		(effects
 			(font
@@
 	(label "SCLK"
 		(at 120.65 153.67 180)
+		(fields_autoplaced yes)
 		(effects
 			(font
@@
 	(label "AV3V3"
 		(at 15.24 175.26 0)
+		(fields_autoplaced yes)
 		(effects
 			(font
@@
 	(label "SATA_RXN"
 		(at 107.95 68.58 180)
+		(fields_autoplaced yes)
 		(effects
 			(font
@@
 	(label "AV1V2"
 		(at 148.59 97.79 180)
+		(fields_autoplaced yes)
 		(effects
 			(font
@@
 	(label "AV3V3"
 		(at 87.63 153.67 0)
+		(fields_autoplaced yes)
 		(effects
 			(font
@@
 	(label "SI"
 		(at 119.38 156.21 180)
+		(fields_autoplaced yes)
 		(effects
 			(font
@@
 	(label "SI"
 		(at 105.41 137.16 90)
+		(fields_autoplaced yes)
 		(effects
 			(font
@@
 	(label "SATA_TXN"
 		(at 102.87 71.12 180)
+		(fields_autoplaced yes)
 		(effects
 			(font
@@
 	(label "AV3V3"
 		(at 73.66 110.49 0)
+		(fields_autoplaced yes)
 		(effects
 			(font
@@
 	(label "SCLK"
 		(at 100.33 137.16 90)
+		(fields_autoplaced yes)
 		(effects
 			(font
@@
 	(label "SATA_TXN"
 		(at 175.26 52.07 180)
+		(fields_autoplaced yes)
 		(effects
 			(font
@@
 	(label "AV1V2"
 		(at 73.66 175.26 180)
+		(fields_autoplaced yes)
 		(effects
 			(font
@@
 	(label "AV1V2"
 		(at 148.59 90.17 180)
+		(fields_autoplaced yes)
 		(effects
 			(font
@@
 	(label "HDD_LED"
 		(at 113.03 137.16 90)
+		(fields_autoplaced yes)
 		(effects
 			(font
@@
 	(label "AV3V3"
 		(at 60.96 73.66 270)
+		(fields_autoplaced yes)
 		(effects
 			(font
@@
 	(label "AV3V3"
 		(at 77.47 92.71 0)
+		(fields_autoplaced yes)
 		(effects
 			(font
@@
 	(label "AV1V2"
 		(at 113.03 71.12 270)
+		(fields_autoplaced yes)
 		(effects
 			(font
@@
 	(label "AV3V3"
 		(at 110.49 137.16 90)
+		(fields_autoplaced yes)
 		(effects
 			(font
@@
 	(label "SATA_RXN"
 		(at 175.26 57.15 180)
+		(fields_autoplaced yes)
 		(effects
 			(font
@@
 	(label "HDD_LED"
 		(at 31.75 148.59 180)
+		(fields_autoplaced yes)
 		(effects
 			(font
@@
 	(label "AV1V2"
 		(at 77.47 95.25 0)
+		(fields_autoplaced yes)
 		(effects
 			(font
@@
 	(label "SO"
 		(at 119.38 158.75 180)
+		(fields_autoplaced yes)
 		(effects
 			(font
@@
 	(label "AV3V3"
 		(at 87.63 156.21 0)
+		(fields_autoplaced yes)
 		(effects
 			(font
@@
 	(label "AV1V2"
 		(at 105.41 71.12 270)
+		(fields_autoplaced yes)
 		(effects
 			(font
@@
 	(label "SATA_TXP"
 		(at 175.26 46.99 180)
+		(fields_autoplaced yes)
 		(effects
 			(font
@@
 	(label "SATA_TXP"
 		(at 100.33 73.66 180)
+		(fields_autoplaced yes)
 		(effects
 			(font
@@
 	(label "AV3V3"
 		(at 158.75 115.57 180)
+		(fields_autoplaced yes)
 		(effects
 			(font
@@
 	(label "AV1V2"
 		(at 102.87 137.16 90)
+		(fields_autoplaced yes)
 		(effects
 			(font
@@
 	(label "AV3V3"
 		(at 105.41 148.59 180)
+		(fields_autoplaced yes)
 		(effects
 			(font
@@
 	(label "AV1V2"
 		(at 49.53 105.41 180)
+		(fields_autoplaced yes)
 		(effects
 			(font
@@
 	(label "SO"
 		(at 97.79 137.16 90)
+		(fields_autoplaced yes)
 		(effects
 			(font
@@
 	(label "AV1V2"
 		(at 148.59 105.41 180)
+		(fields_autoplaced yes)
 		(effects
 			(font
@@
 	(label "CS"
 		(at 91.44 158.75 0)
+		(fields_autoplaced yes)
 		(effects
 			(font
@@
 	(label "AV1V2"
 		(at 118.11 137.16 90)
+		(fields_autoplaced yes)
 		(effects
 			(font
@@
 		(shape output)
 		(at 132.08 92.71 0)
+		(fields_autoplaced yes)
+		(effects
+			(font
+				(size 1.27 1.27)
+			)
+			(justify left)
+		)
+	)
+	(hierarchical_label "VBUS"
+		(shape input)
+		(at 67.31 102.87 0)
+		(fields_autoplaced yes)
 		(effects
 			(font
@@
 		(shape bidirectional)
 		(at 132.08 113.03 0)
+		(fields_autoplaced yes)
 		(effects
 			(font
@@
 		(shape output)
 		(at 132.08 95.25 0)
+		(fields_autoplaced yes)
 		(effects
 			(font
@@
 		(shape input)
 		(at 132.08 100.33 0)
+		(fields_autoplaced yes)
 		(effects
 			(font
@@
 		(shape bidirectional)
 		(at 132.08 118.11 0)
+		(fields_autoplaced yes)
 		(effects
 			(font
@@
 		(shape input)
 		(at 132.08 102.87 0)
+		(fields_autoplaced yes)
+		(effects
+			(font
+				(size 1.27 1.27)
+			)
+			(justify left)
+		)
+	)
+	(hierarchical_label "VBUS"
+		(shape input)
+		(at 135.89 128.27 0)
+		(fields_autoplaced yes)
 		(effects
 			(font
@@
 	)
 	(symbol
-		(lib_id "power:+5V")
-		(at 67.31 102.87 0)
-		(unit 1)
-		(exclude_from_sim no)
-		(in_bom yes)
-		(on_board yes)
-		(dnp no)
-		(fields_autoplaced yes)
-		(property "Reference" "#PWR0804"
-			(at 67.31 106.68 0)
-			(effects
-				(font
-					(size 1.27 1.27)
-				)
-				(hide yes)
-			)
-		)
-		(property "Value" "+5V"
-			(at 67.31 97.79 0)
-			(effects
-				(font
-					(size 1.27 1.27)
-				)
-			)
-		)
-		(property "Footprint" ""
-			(at 67.31 102.87 0)
-			(effects
-				(font
-					(size 1.27 1.27)
-				)
-				(hide yes)
-			)
-		)
-		(property "Datasheet" ""
-			(at 67.31 102.87 0)
-			(effects
-				(font
-					(size 1.27 1.27)
-				)
-				(hide yes)
-			)
-		)
-		(property "Description" "Power symbol creates a global label with name \"+5V\""
-			(at 67.31 102.87 0)
-			(effects
-				(font
-					(size 1.27 1.27)
-				)
-				(hide yes)
-			)
-		)
-		(pin "1"
-		)
-		(instances
-			(project "mainboard4"
-				(path "/dd07ab80-a59c-44f4-ac7d-849e21e1384e/5db2a135-33ff-4812-ab9d-2394338dfef8"
-					(reference "#PWR0804")
-					(unit 1)
-				)
-			)
-		)
-	)
-	(symbol
 		(lib_id "Device:C")
 		(at 135.89 132.08 0)
@@
 					(unit 1)
 				)
-			)
-		)
-	)
-	(symbol
-		(lib_id "power:+5V")
-		(at 135.89 128.27 0)
-		(unit 1)
-		(exclude_from_sim no)
-		(in_bom yes)
-		(on_board yes)
-		(dnp no)
-		(fields_autoplaced yes)
-		(property "Reference" "#PWR0805"
-			(at 135.89 132.08 0)
-			(effects
-				(font
-					(size 1.27 1.27)
-				)
-				(hide yes)
-			)
-		)
-		(property "Value" "+5V"
-			(at 135.89 123.19 0)
-			(effects
-				(font
-					(size 1.27 1.27)
-				)
-			)
-		)
-		(property "Footprint" ""
-			(at 135.89 128.27 0)
-			(effects
-				(font
-					(size 1.27 1.27)
-				)
-				(hide yes)
-			)
-		)
-		(property "Datasheet" ""
-			(at 135.89 128.27 0)
-			(effects
-				(font
-					(size 1.27 1.27)
-				)
-				(hide yes)
-			)
-		)
-		(property "Description" "Power symbol creates a global label with name \"+5V\""
-			(at 135.89 128.27 0)
-			(effects
-				(font
-					(size 1.27 1.27)
-				)
-				(hide yes)
-			)
-		)
-		(pin "1"
-		)
-		(instances
-			(project "mainboard4"
-				(path "/dd07ab80-a59c-44f4-ac7d-849e21e1384e/5db2a135-33ff-4812-ab9d-2394338dfef8"
-					(reference "#PWR0805")
-					(unit 1)
-				)

Commit message: end route
Parts:
- removed C101: 0.1uF, Capacitor_SMD:C_0402_1005Metric_Pad0.74x0.62mm_HandSolder, symbol Device:C
- renumbered C75 to C68, C80 to C69, C78 to C70, C72 to C71, C90 to C72, C70 to C73, C92 to C75, C91 to C77, C69 to C78, C68 to C81, C103 to C88, C71 to C89, C93 to C90, C89 to C91, C81 to C94, C76 to C95, C77 to C96, C79 to C97, R51 to R50, R58 to R51
Other:
- moved on the sheet: C75, C91
