File: PHY.kicad_sch (KiCad schematic)
At the start: 29 parts, among them U13 LAN8742A, Y3 25Mhz

Commit message: add logp
Parts:
- renumbered R29 to R26, R31 to R28, R32 to R29, R33 to R30, R34 to R31, R35 to R32, R36 to R33, R37 to R34, R42 to R39, R43 to R40, R44 to R41, R45 to R42, R46 to R43, R47 to R44, R48 to R45, R51 to R48, R52 to R49
Changed lines of the file:
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@@
 		(shape input)
 		(at 78.74 116.84 180)
-		(fields_autoplaced yes)
 		(effects
 			(font
@@
 		(shape output)
 		(at 217.17 121.92 0)
-		(fields_autoplaced yes)
 		(effects
 			(font
@@
 		(shape output)
 		(at 78.74 109.22 180)
-		(fields_autoplaced yes)
 		(effects
 			(font
@@
 		(shape input)
 		(at 78.74 114.3 180)
-		(fields_autoplaced yes)
 		(effects
 			(font
@@
 		(shape output)
 		(at 217.17 134.62 0)
-		(fields_autoplaced yes)
 		(effects
 			(font
@@
 		(shape input)
 		(at 217.17 106.68 0)
-		(fields_autoplaced yes)
 		(effects
 			(font
@@
 		(shape output)
 		(at 217.17 116.84 0)
-		(fields_autoplaced yes)
 		(effects
 			(font
@@
 		(shape input)
 		(at 217.17 109.22 0)
-		(fields_autoplaced yes)
 		(effects
 			(font
@@
 		(shape input)
 		(at 217.17 127 0)
-		(fields_autoplaced yes)
 		(effects
 			(font
@@
 		(shape input)
 		(at 217.17 132.08 0)
-		(fields_autoplaced yes)
 		(effects
 			(font
@@
 		(shape output)
 		(at 217.17 114.3 0)
-		(fields_autoplaced yes)
 		(effects
 			(font
@@
 		(shape input)
 		(at 217.17 111.76 0)
-		(fields_autoplaced yes)
 		(effects
 			(font
@@
 		(shape bidirectional)
 		(at 217.17 124.46 0)
-		(fields_autoplaced yes)
 		(effects
 			(font
@@
 		(shape output)
 		(at 78.74 111.76 180)
-		(fields_autoplaced yes)
 		(effects
 			(font
@@
 		(on_board yes)
 		(dnp no)
-		(property "Reference" "R46"
+		(property "Reference" "R43"
 			(at 206.502 115.57 90)
 			(effects
@@
 			(project "mainboard4"
 				(path "/dd07ab80-a59c-44f4-ac7d-849e21e1384e/4fc6aed4-b6ec-46a7-b9d1-1f9060000df7"
-					(reference "R46")
+					(reference "R43")
 					(unit 1)
 				)
@@
 		(on_board yes)
 		(dnp no)
-		(property "Reference" "R44"
+		(property "Reference" "R41"
 			(at 94.488 92.456 0)
 			(effects
@@
 			(project "mainboard4"
 				(path "/dd07ab80-a59c-44f4-ac7d-849e21e1384e/4fc6aed4-b6ec-46a7-b9d1-1f9060000df7"
-					(reference "R44")
+					(reference "R41")
 					(unit 1)
 				)
@@
 		(on_board yes)
 		(dnp no)
-		(property "Reference" "R47"
+		(property "Reference" "R44"
 			(at 82.042 129.032 0)
 			(effects
@@
 			(project "mainboard4"
 				(path "/dd07ab80-a59c-44f4-ac7d-849e21e1384e/4fc6aed4-b6ec-46a7-b9d1-1f9060000df7"
-					(reference "R47")
+					(reference "R44")
 					(unit 1)
 				)
@@
 		(on_board yes)
 		(dnp no)
-		(property "Reference" "R37"
+		(property "Reference" "R34"
 			(at 76.962 90.932 0)
 			(effects
@@
 			(project "mainboard4"
 				(path "/dd07ab80-a59c-44f4-ac7d-849e21e1384e/4fc6aed4-b6ec-46a7-b9d1-1f9060000df7"
-					(reference "R37")
+					(reference "R34")
 					(unit 1)
 				)
@@
 		(on_board yes)
 		(dnp no)
-		(property "Reference" "R43"
+		(property "Reference" "R40"
 			(at 206.756 113.03 90)
 			(effects
@@
 			(project "mainboard4"
 				(path "/dd07ab80-a59c-44f4-ac7d-849e21e1384e/4fc6aed4-b6ec-46a7-b9d1-1f9060000df7"
-					(reference "R43")
+					(reference "R40")
 					(unit 1)
 				)
@@
 		(on_board yes)
 		(dnp no)
-		(property "Reference" "R42"
+		(property "Reference" "R39"
 			(at 104.902 93.218 0)
 			(effects
@@
 			(project "mainboard4"
 				(path "/dd07ab80-a59c-44f4-ac7d-849e21e1384e/4fc6aed4-b6ec-46a7-b9d1-1f9060000df7"
-					(reference "R42")
+					(reference "R39")
 					(unit 1)
 				)
@@
 		(on_board yes)
 		(dnp no)
-		(property "Reference" "R36"
+		(property "Reference" "R33"
 			(at 235.204 121.412 0)
 			(effects
@@
 			(project "mainboard4"
 				(path "/dd07ab80-a59c-44f4-ac7d-849e21e1384e/4fc6aed4-b6ec-46a7-b9d1-1f9060000df7"
-					(reference "R36")
+					(reference "R33")
 					(unit 1)
 				)
@@
 		(on_board yes)
 		(dnp no)
-		(property "Reference" "R35"
+		(property "Reference" "R32"
 			(at 86.106 92.202 0)
 			(effects
@@
 			(project "mainboard4"
 				(path "/dd07ab80-a59c-44f4-ac7d-849e21e1384e/4fc6aed4-b6ec-46a7-b9d1-1f9060000df7"
-					(reference "R35")
+					(reference "R32")
 					(unit 1)
 				)
@@
 		(on_board yes)
 		(dnp no)
-		(property "Reference" "R48"
+		(property "Reference" "R45"
 			(at 179.832 92.964 0)
 			(effects
@@
 			(project "mainboard4"
 				(path "/dd07ab80-a59c-44f4-ac7d-849e21e1384e/4fc6aed4-b6ec-46a7-b9d1-1f9060000df7"
-					(reference "R48")
+					(reference "R45")
 					(unit 1)
 				)
@@
 		(dnp no)
 		(fields_autoplaced yes)
-		(property "Reference" "R51"
+		(property "Reference" "R48"
 			(at 104.775 142.875 0)
 			(effects
@@
 			(project "mainboard4"
 				(path "/dd07ab80-a59c-44f4-ac7d-849e21e1384e/4fc6aed4-b6ec-46a7-b9d1-1f9060000df7"
-					(reference "R51")
+					(reference "R48")
 					(unit 1)
 				)
@@
 		(on_board yes)
 		(dnp no)
-		(property "Reference" "R45"
+		(property "Reference" "R42"
 			(at 172.212 92.964 0)
 			(effects
@@
 			(project "mainboard4"
 				(path "/dd07ab80-a59c-44f4-ac7d-849e21e1384e/4fc6aed4-b6ec-46a7-b9d1-1f9060000df7"
-					(reference "R45")
+					(reference "R42")
 					(unit 1)
 				)
@@
 		(on_board yes)
 		(dnp no)
-		(property "Reference" "R29"
+		(property "Reference" "R26"
 			(at 194.31 92.964 0)
 			(effects
@@
 			(project "mainboard4"
 				(path "/dd07ab80-a59c-44f4-ac7d-849e21e1384e/4fc6aed4-b6ec-46a7-b9d1-1f9060000df7"
-					(reference "R29")
+					(reference "R26")
 					(unit 1)
 				)
@@
 		(dnp no)
 		(fields_autoplaced yes)
-		(property "Reference" "R52"
+		(property "Reference" "R49"
 			(at 115.57 142.875 0)
 			(effects
@@
 			(project "mainboard4"
 				(path "/dd07ab80-a59c-44f4-ac7d-849e21e1384e/4fc6aed4-b6ec-46a7-b9d1-1f9060000df7"
-					(reference "R52")
+					(reference "R49")
 					(unit 1)
 				)
@@
 		(on_board yes)
 		(dnp no)
-		(property "Reference" "R31"
+		(property "Reference" "R28"
 			(at 213.36 135.89 90)
 			(effects
@@
 			(project "mainboard4"
 				(path "/dd07ab80-a59c-44f4-ac7d-849e21e1384e/4fc6aed4-b6ec-46a7-b9d1-1f9060000df7"
-					(reference "R31")
+					(reference "R28")
 					(unit 1)
 				)
@@
 		(on_board yes)
 		(dnp no)
-		(property "Reference" "R33"
+		(property "Reference" "R30"
 			(at 187.198 92.964 0)
 			(effects
@@
 			(project "mainboard4"
 				(path "/dd07ab80-a59c-44f4-ac7d-849e21e1384e/4fc6aed4-b6ec-46a7-b9d1-1f9060000df7"
-					(reference "R33")
+					(reference "R30")
 					(unit 1)
 				)
@@
 		(on_board yes)
 		(dnp no)
-		(property "Reference" "R32"
+		(property "Reference" "R29"
 			(at 203.2 92.964 0)
 			(effects
@@
 			(project "mainboard4"
 				(path "/dd07ab80-a59c-44f4-ac7d-849e21e1384e/4fc6aed4-b6ec-46a7-b9d1-1f9060000df7"
-					(reference "R32")
+					(reference "R29")
 					(unit 1)
 				)
@@
 		(on_board yes)
 		(dnp no)
-		(property "Reference" "R34"
+		(property "Reference" "R31"
 			(at 206.502 120.65 90)
 			(effects
@@
 			(project "mainboard4"
 				(path "/dd07ab80-a59c-44f4-ac7d-849e21e1384e/4fc6aed4-b6ec-46a7-b9d1-1f9060000df7"
-					(reference "R34")
+					(reference "R31")
 					(unit 1)
 				)
