File: PHY.kicad_sch (KiCad schematic)
At the start: 29 parts, among them U13 LAN8742A, Y3 25Mhz

Commit message: end route
Parts:
- renumbered FB3 to FB2
Changed lines of the file:
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@@
 		(on_board yes)
 		(dnp no)
-		(property "Reference" "FB3"
+		(property "Reference" "FB2"
 			(at 124.206 68.072 0)
 			(effects
@@
 			(project "mainboard4"
 				(path "/dd07ab80-a59c-44f4-ac7d-849e21e1384e/4fc6aed4-b6ec-46a7-b9d1-1f9060000df7"
-					(reference "FB3")
+					(reference "FB2")
 					(unit 1)
 				)

Commit message: データをアップロード
Parts:
- added C56, C57, C58, C59: 0.1μF, Capacitor_SMD:C_0402_1005Metric_Pad0.74x0.62mm_HandSolder, symbol Device:C_Small
- added R27: 10k, Resistor_SMD:R_0603_1608Metric_Pad0.98x0.95mm_HandSolder, symbol Device:R
- C50: renamed from C61; footprint Capacitor_SMD:C_0603_1608Metric_Pad1.08x0.95mm_HandSolder -> Capacitor_SMD:C_0402_1005Metric_Pad0.74x0.62mm_HandSolder
- C51: renamed from C60; footprint Capacitor_SMD:C_0603_1608Metric_Pad1.08x0.95mm_HandSolder -> Capacitor_SMD:C_0402_1005Metric_Pad0.74x0.62mm_HandSolder
- R14: renamed from R29; footprint Resistor_SMD:R_0603_1608Metric_Pad0.98x0.95mm_HandSolder -> Resistor_SMD:R_0402_1005Metric_Pad0.72x0.64mm_HandSolder
- R15: renamed from R28; footprint Resistor_SMD:R_0603_1608Metric_Pad0.98x0.95mm_HandSolder -> Resistor_SMD:R_0402_1005Metric_Pad0.72x0.64mm_HandSolder
- R17: renamed from R26; footprint Resistor_SMD:R_0603_1608Metric_Pad0.98x0.95mm_HandSolder -> Resistor_SMD:R_0402_1005Metric_Pad0.72x0.64mm_HandSolder
- R18: renamed from R31; footprint Resistor_SMD:R_0603_1608Metric_Pad0.98x0.95mm_HandSolder -> Resistor_SMD:R_0402_1005Metric_Pad0.72x0.64mm_HandSolder
- R19: renamed from R32; footprint Resistor_SMD:R_0603_1608Metric_Pad0.98x0.95mm_HandSolder -> Resistor_SMD:R_0402_1005Metric_Pad0.72x0.64mm_HandSolder
- R20: renamed from R48; value 1k -> 200
- R21: renamed from R30; footprint Resistor_SMD:R_0603_1608Metric_Pad0.98x0.95mm_HandSolder -> Resistor_SMD:R_0402_1005Metric_Pad0.72x0.64mm_HandSolder
- R22: renamed from R33; footprint Resistor_SMD:R_0603_1608Metric_Pad0.98x0.95mm_HandSolder -> Resistor_SMD:R_0402_1005Metric_Pad0.72x0.64mm_HandSolder
- R23: renamed from R34; footprint Resistor_SMD:R_0603_1608Metric_Pad0.98x0.95mm_HandSolder -> Resistor_SMD:R_0402_1005Metric_Pad0.72x0.64mm_HandSolder
- R24: renamed from R49; value 1k -> 200
- R25: renamed from R39; footprint Resistor_SMD:R_0603_1608Metric_Pad0.98x0.95mm_HandSolder -> Resistor_SMD:R_0402_1005Metric_Pad0.72x0.64mm_HandSolder
- R26: renamed from R42; footprint Resistor_SMD:R_0603_1608Metric_Pad0.98x0.95mm_HandSolder -> Resistor_SMD:R_0402_1005Metric_Pad0.72x0.64mm_HandSolder
- R28: renamed from R41; footprint Resistor_SMD:R_0603_1608Metric_Pad0.98x0.95mm_HandSolder -> Resistor_SMD:R_0402_1005Metric_Pad0.72x0.64mm_HandSolder
- R29: renamed from R40; footprint Resistor_SMD:R_0603_1608Metric_Pad0.98x0.95mm_HandSolder -> Resistor_SMD:R_0402_1005Metric_Pad0.72x0.64mm_HandSolder
- R32: renamed from R43; footprint Resistor_SMD:R_0603_1608Metric_Pad0.98x0.95mm_HandSolder -> Resistor_SMD:R_0402_1005Metric_Pad0.72x0.64mm_HandSolder
- R33: renamed from R45; footprint Resistor_SMD:R_0603_1608Metric_Pad0.98x0.95mm_HandSolder -> Resistor_SMD:R_0402_1005Metric_Pad0.72x0.64mm_HandSolder
- renumbered C54 to C44, C59 to C48, C53 to C49, C57 to C52, C56 to C53, D9 to D4, D8 to D5, R44 to R34, U13 to U9, Y3 to Y2
Connections:
- net GND: now also R27.2
- net at R24.1, U9.2 (LED2/~{INTSEL}): now also R27.1
- net RXN renamed RXC_N
- net RXC_N: now also C56.2
- net RXP renamed RXC_P
- net RXC_P: now also C57.2
- net TXN renamed TXC_N
- net TXC_N: now also C58.2
- net TXP renamed TXC_P
- net TXC_P: now also C59.2
- new net TRD0_N: C56.1
- new net TRD0_P: C57.1
- new net TRD1_N: C58.1
- new net TRD1_P: C59.1
Other:
- moved on the sheet: C44, C50, C51, C52, C53, D4, D5, R20, R22, R24, Y2
