File: USB2Ethernet.kicad_sch (KiCad schematic)
At the start: 36 parts, among them U16 LAN9514, U19 CAT250xxx, Y6 25Mhz

Commit message: change USB2.0
Parts:
- removed R57: 400kΩ, Resistor_SMD:R_0603_1608Metric_Pad0.98x0.95mm_HandSolder, symbol Device:R
- added J16: USB_A_Stacked, Connector_USB:USB_A_Wuerth_61400826021_Horizontal_Stacked, symbol Connector:USB_A_Stacked
Connections:
- net GND: now also R59.1
- new net VBUS: J16.1 (VBUS1), J16.5 (VBUS2)
Other:
- moved on the sheet: C100, C106, C111, C112, C121, C122, C123, C127, C128, C129, C132, C133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

Commit message: add usb2.0 line
Parts:
- removed C127: 0.01uF, Capacitor_SMD:C_0402_1005Metric_Pad0.74x0.62mm_HandSolder, symbol Device:C
- removed R63: 1k, Resistor_SMD:R_0603_1608Metric_Pad0.98x0.95mm_HandSolder, symbol Device:R
- removed R64: 10kΩ, Resistor_SMD:R_0603_1608Metric_Pad0.98x0.95mm_HandSolder, symbol Device:R
Connections:
- net +3.3V: now also U16.11 (VBUS_DET)
- net GND: now also J16.4 (GND1), J16.8 (GND2)
- net RESET: now reaches U16.12 (~{RESET})
- net USB4DN: now reaches U16.6 (USBDM4)
- net USB4DN: now also J16.6 (D2-)
- net USB4DP: now reaches U16.7 (USBDP4)
- net USB4DP: now also J16.7 (D2+)
- net USB5DN: now reaches U16.8 (USBDM5)
- net USB5DN: now also J16.2 (D1-)
- net USB5DP: now reaches U16.9 (USBDP5)
- net USB5DP: now also J16.3 (D1+)

Commit message: add HDD_LED[
Connections:
- net GND: now also J16.9 (Shield)
Changed lines of the file:
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@@
+	(wire
+		(pts
+			(xy 269.24 113.03) (xy 271.78 113.03)
+		)
+		(stroke
+			(width 0)
+			(type default)
+		)
+	)
 	(wire
 		(pts
@@
 	(label "SI"
 		(at 113.03 81.28 180)
-		(fields_autoplaced yes)
 		(effects
 			(font
@@
 	(label "1.8V"
 		(at 92.71 45.72 180)
-		(fields_autoplaced yes)
 		(effects
 			(font
@@
 	(label "USB5DN"
 		(at 259.08 97.79 180)
-		(fields_autoplaced yes)
 		(effects
 			(font
@@
 	(label "USB4DN"
 		(at 259.08 102.87 180)
-		(fields_autoplaced yes)
 		(effects
 			(font
@@
 	(label "USB4DP"
 		(at 184.15 80.01 180)
-		(fields_autoplaced yes)
 		(effects
 			(font
@@
 	(label "USB5DP"
 		(at 184.15 90.17 180)
-		(fields_autoplaced yes)
 		(effects
 			(font
@@
 	(label "SO"
 		(at 68.58 26.67 180)
-		(fields_autoplaced yes)
 		(effects
 			(font
@@
 	(label "VDDA"
 		(at 87.63 48.26 180)
-		(fields_autoplaced yes)
 		(effects
 			(font
@@
 	(label "CS"
 		(at 36.83 26.67 0)
-		(fields_autoplaced yes)
 		(effects
 			(font
@@
 	(label "SCLK"
 		(at 69.85 21.59 180)
-		(fields_autoplaced yes)
 		(effects
 			(font
@@
 	(label "USB5DN"
 		(at 184.15 92.71 180)
-		(fields_autoplaced yes)
 		(effects
 			(font
@@
 	(label "CS"
 		(at 113.03 76.2 180)
-		(fields_autoplaced yes)
 		(effects
 			(font
@@
 	(label "USB4DN"
 		(at 184.15 82.55 180)
-		(fields_autoplaced yes)
 		(effects
 			(font
@@
 	(label "VDDA"
 		(at 101.6 146.05 0)
-		(fields_autoplaced yes)
 		(effects
 			(font
@@
 	(label "USB4DP"
 		(at 259.08 100.33 180)
-		(fields_autoplaced yes)
 		(effects
 			(font
@@
 	(label "VDDIO"
 		(at 82.55 50.8 180)
-		(fields_autoplaced yes)
 		(effects
 			(font
@@
 	(label "SCLK"
 		(at 114.3 73.66 180)
-		(fields_autoplaced yes)
 		(effects
 			(font
@@
 	(label "1.8V"
 		(at 88.9 127 180)
-		(fields_autoplaced yes)
 		(effects
 			(font
@@
 	(label "SI"
 		(at 68.58 24.13 180)
-		(fields_autoplaced yes)
 		(effects
 			(font
@@
 	(label "SO"
 		(at 113.03 78.74 180)
-		(fields_autoplaced yes)
 		(effects
 			(font
@@
 	(label "VDDA"
 		(at 193.04 83.82 180)
-		(fields_autoplaced yes)
 		(effects
 			(font
@@
 	(label "VDDIO"
 		(at 90.17 168.91 0)
-		(fields_autoplaced yes)
 		(effects
 			(font
@@
 	(label "USB5DP"
 		(at 259.08 95.25 180)
-		(fields_autoplaced yes)
 		(effects
 			(font
@@
 		(shape bidirectional)
 		(at 175.26 59.69 0)
-		(fields_autoplaced yes)
 		(effects
 			(font
@@
 		(shape bidirectional)
 		(at 175.26 69.85 0)
-		(fields_autoplaced yes)
 		(effects
 			(font
@@
 		(shape input)
 		(at 259.08 87.63 180)
-		(fields_autoplaced yes)
 		(effects
 			(font
@@
 		(shape output)
 		(at 226.06 102.87 0)
-		(fields_autoplaced yes)
 		(effects
 			(font
@@
 		(shape input)
 		(at 226.06 110.49 0)
-		(fields_autoplaced yes)
 		(effects
 			(font
@@
 		(shape bidirectional)
 		(at 175.26 72.39 0)
-		(fields_autoplaced yes)
 		(effects
 			(font
@@
 		(shape bidirectional)
 		(at 175.26 62.23 0)
-		(fields_autoplaced yes)
 		(effects
 			(font
@@
 		(shape input)
 		(at 226.06 107.95 0)
-		(fields_autoplaced yes)
 		(effects
 			(font
@@
 		(shape input)
 		(at 73.66 68.58 180)
-		(fields_autoplaced yes)
 		(effects
 			(font
@@
 		(shape output)
 		(at 226.06 100.33 0)
-		(fields_autoplaced yes)
 		(effects
 			(font
@@
 		(shape input)
 		(at 144.78 59.69 180)
-		(fields_autoplaced yes)
 		(effects
 			(font
@@
 		(shape input)
 		(at 144.78 62.23 180)
-		(fields_autoplaced yes)
-		(effects
-			(font
+		(effects
+			(font

Commit message: end route
Parts:
- renumbered C122 to C100, C121 to C101, C123 to C102, C128 to C103, C129 to C104, C133 to C105, C132 to C106, C134 to C107, C87 to C74, C88 to C76, C95 to C82, C96 to C83, C97 to C84, C98 to C85, C99 to C86, C100 to C87, C106 to C92, C111 to C93, C112 to C99, FB4 to FB3, FB5 to FB4, J16 to J8, R59 to R56, R61 to R57, R62 to R58, R68 to R59, U19 to U17, Y6 to Y5
Changed lines of the file:
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@@
 		(dnp no)
 		(fields_autoplaced yes)
-		(property "Reference" "C97"
+		(property "Reference" "C84"
 			(at 105.41 148.5899 0)
 			(effects
@@
 			(project "mainboard4"
 				(path "/dd07ab80-a59c-44f4-ac7d-849e21e1384e/3546f414-4018-45c7-a00a-bf02d214bf7f"
-					(reference "C97")
+					(reference "C84")
 					(unit 1)
 				)
@@
 		(dnp no)
 		(fields_autoplaced yes)
-		(property "Reference" "C132"
+		(property "Reference" "C106"
 			(at 46.99 171.4499 0)
 			(effects
@@
 			(project "mainboard4"
 				(path "/dd07ab80-a59c-44f4-ac7d-849e21e1384e/3546f414-4018-45c7-a00a-bf02d214bf7f"
-					(reference "C132")
+					(reference "C106")
 					(unit 1)
 				)
@@
 		(dnp no)
 		(fields_autoplaced yes)
-		(property "Reference" "C96"
+		(property "Reference" "C83"
 			(at 92.71 148.5899 0)
 			(effects
@@
 			(project "mainboard4"
 				(path "/dd07ab80-a59c-44f4-ac7d-849e21e1384e/3546f414-4018-45c7-a00a-bf02d214bf7f"
-					(reference "C96")
+					(reference "C83")
 					(unit 1)
 				)
@@
 		(on_board yes)
 		(dnp no)
-		(property "Reference" "C87"
+		(property "Reference" "C74"
 			(at 35.306 121.666 0)
 			(effects
@@
 			(project "mainboard4"
 				(path "/dd07ab80-a59c-44f4-ac7d-849e21e1384e/3546f414-4018-45c7-a00a-bf02d214bf7f"
-					(reference "C87")
+					(reference "C74")
 					(unit 1)
 				)
@@
 		(dnp no)
 		(fields_autoplaced yes)
-		(property "Reference" "R62"
+		(property "Reference" "R58"
 			(at 128.27 93.98 90)
 			(effects
@@
 			(project "mainboard4"
 				(path "/dd07ab80-a59c-44f4-ac7d-849e21e1384e/3546f414-4018-45c7-a00a-bf02d214bf7f"
-					(reference "R62")
+					(reference "R58")
 					(unit 1)
 				)
@@
 		(dnp no)
 		(fields_autoplaced yes)
-		(property "Reference" "C98"
+		(property "Reference" "C85"
 			(at 80.01 148.5899 0)
 			(effects
@@
 			(project "mainboard4"
 				(path "/dd07ab80-a59c-44f4-ac7d-849e21e1384e/3546f414-4018-45c7-a00a-bf02d214bf7f"
-					(reference "C98")
+					(reference "C85")
 					(unit 1)
 				)
@@
 		(on_board yes)
 		(dnp no)
-		(property "Reference" "Y6"
+		(property "Reference" "Y5"
 			(at 38.1 113.0614 0)
 			(effects
@@
 			(project "mainboard4"
 				(path "/dd07ab80-a59c-44f4-ac7d-849e21e1384e/3546f414-4018-45c7-a00a-bf02d214bf7f"
-					(reference "Y6")
+					(reference "Y5")
 					(unit 1)
 				)
@@
 		(dnp no)
 		(fields_autoplaced yes)
-		(property "Reference" "U19"
+		(property "Reference" "U17"
 			(at 56.8041 13.97 0)
 			(effects
@@
 			(project "mainboard4"
 				(path "/dd07ab80-a59c-44f4-ac7d-849e21e1384e/3546f414-4018-45c7-a00a-bf02d214bf7f"
-					(reference "U19")
+					(reference "U17")
 					(unit 1)
 				)
@@
 		(dnp no)
 		(fields_autoplaced yes)
-		(property "Reference" "C106"
+		(property "Reference" "C92"
 			(at 100.33 35.5599 0)
 			(effects
@@
 			(project "mainboard4"
 				(path "/dd07ab80-a59c-44f4-ac7d-849e21e1384e/3546f414-4018-45c7-a00a-bf02d214bf7f"
-					(reference "C106")
+					(reference "C92")
 					(unit 1)
 				)
@@
 		(dnp no)
 		(fields_autoplaced yes)
-		(property "Reference" "C122"
+		(property "Reference" "C100"
 			(at 59.69 171.4499 0)
 			(effects
@@
 			(project "mainboard4"
 				(path "/dd07ab80-a59c-44f4-ac7d-849e21e1384e/3546f414-4018-45c7-a00a-bf02d214bf7f"
-					(reference "C122")
+					(reference "C100")
 					(unit 1)
 				)
@@
 		(dnp no)
 		(fields_autoplaced yes)
-		(property "Reference" "R68"
+		(property "Reference" "R59"
 			(at 44.45 29.2099 0)
 			(effects
@@
 			(project "mainboard4"
 				(path "/dd07ab80-a59c-44f4-ac7d-849e21e1384e/3546f414-4018-45c7-a00a-bf02d214bf7f"
-					(reference "R68")
+					(reference "R59")
 					(unit 1)
 				)
@@
 		(dnp no)
 		(fields_autoplaced yes)
-		(property "Reference" "C111"
+		(property "Reference" "C93"
 			(at 72.39 171.4499 0)
 			(effects
@@
 			(project "mainboard4"
 				(path "/dd07ab80-a59c-44f4-ac7d-849e21e1384e/3546f414-4018-45c7-a00a-bf02d214bf7f"
-					(reference "C111")
+					(reference "C93")
 					(unit 1)
 				)
@@
 		(dnp no)
 		(fields_autoplaced yes)
-		(property "Reference" "C128"
+		(property "Reference" "C103"
 			(at 92.71 129.5399 0)
 			(effects
@@
 			(project "mainboard4"
 				(path "/dd07ab80-a59c-44f4-ac7d-849e21e1384e/3546f414-4018-45c7-a00a-bf02d214bf7f"
-					(reference "C128")
+					(reference "C103")
 					(unit 1)
 				)
@@
 		(dnp no)
 		(fields_autoplaced yes)
-		(property "Reference" "FB5"
+		(property "Reference" "FB4"
 			(at 25.3492 138.43 90)
 			(effects
@@
 			(project "mainboard4"
 				(path "/dd07ab80-a59c-44f4-ac7d-849e21e1384e/3546f414-4018-45c7-a00a-bf02d214bf7f"
-					(reference "FB5")
+					(reference "FB4")
 					(unit 1)
 				)
@@
 		(dnp no)
 		(fields_autoplaced yes)
-		(property "Reference" "C133"
+		(property "Reference" "C105"
 			(at 38.1 171.4499 0)
 			(effects
@@
 			(project "mainboard4"
 				(path "/dd07ab80-a59c-44f4-ac7d-849e21e1384e/3546f414-4018-45c7-a00a-bf02d214bf7f"
-					(reference "C133")
+					(reference "C105")
 					(unit 1)
 				)
@@
 		(dnp no)
 		(fields_autoplaced yes)
-		(property "Reference" "C129"
+		(property "Reference" "C104"
 			(at 85.09 171.4499 0)
 			(effects
@@
 			(project "mainboard4"
 				(path "/dd07ab80-a59c-44f4-ac7d-849e21e1384e/3546f414-4018-45c7-a00a-bf02d214bf7f"
-					(reference "C129")
+					(reference "C104")
 					(unit 1)
 				)
@@
 		(dnp no)
 		(fields_autoplaced yes)
-		(property "Reference" "C99"
+		(property "Reference" "C86"
 			(at 58.42 148.5899 0)
 			(effects
@@
 			(project "mainboard4"
 				(path "/dd07ab80-a59c-44f4-ac7d-849e21e1384e/3546f414-4018-45c7-a00a-bf02d214bf7f"
-					(reference "C99")
+					(reference "C86")
 					(unit 1)
 				)
@@
 		(on_board yes)
 		(dnp no)
-		(property "Reference" "J16"
+		(property "Reference" "J8"
 			(at 269.24 80.01 0)
 			(effects
@@
 			(project ""
 				(path "/dd07ab80-a59c-44f4-ac7d-849e21e1384e/3546f414-4018-45c7-a00a-bf02d214bf7f"
-					(reference "J16")
+					(reference "J8")
 					(unit 1)
 				)
@@
 		(dnp no)
 		(fields_autoplaced yes)
-		(property "Reference" "C95"
+		(property "Reference" "C82"
 			(at 71.12 148.5899 0)
 			(effects
@@
 			(project "mainboard4"
 				(path "/dd07ab80-a59c-44f4-ac7d-849e21e1384e/3546f414-4018-45c7-a00a-bf02d214bf7f"
-					(reference "C95")
+					(reference "C82")
 					(unit 1)
 				)
@@
 		(dnp no)
 		(fields_autoplaced yes)
-		(property "Reference" "R59"
+		(property "Reference" "R56"
 			(at 138.43 102.87 90)
 			(effects
@@
 			(project "mainboard4"
 				(path "/dd07ab80-a59c-44f4-ac7d-849e21e1384e/3546f414-4018-45c7-a00a-bf02d214bf7f"
-					(reference "R59")
+					(reference "R56")
 					(unit 1)
 				)
@@
 		(on_board yes)
 		(dnp no)
-		(property "Reference" "C88"
+		(property "Reference" "C76"
 			(at 71.12 121.9199 0)
 			(effects
@@
 			(project "mainboard4"
 				(path "/dd07ab80-a59c-44f4-ac7d-849e21e1384e/3546f414-4018-45c7-a00a-bf02d214bf7f"
-					(reference "C88")
+					(reference "C76")
 					(unit 1)
 				)
@@
 		(dnp no)
 		(fields_autoplaced yes)
-		(property "Reference" "C123"
+		(property "Reference" "C102"
 			(at 105.41 129.5399 0)
 			(effects
@@
 			(project "mainboard4"
 				(path "/dd07ab80-a59c-44f4-ac7d-849e21e1384e/3546f414-4018-45c7-a00a-bf02d214bf7f"
-					(reference "C123")
+					(reference "C102")
 					(unit 1)
 				)
@@
 		(dnp no)
 		(fields_autoplaced yes)
-		(property "Reference" "C112"
+		(property "Reference" "C99"
 			(at 36.83 148.5899 0)
 			(effects
@@
 			(project "mainboard4"
 				(path "/dd07ab80-a59c-44f4-ac7d-849e21e1384e/3546f414-4018-45c7-a00a-bf02d214bf7f"
-					(reference "C112")
+					(reference "C99")
 					(unit 1)
 				)
@@
 		(on_board yes)
 		(dnp no)
-		(property "Reference" "FB4"
+		(property "Reference" "FB3"
 			(at 103.632 27.178 90)
 			(effects
@@
 			(project "mainboard4"
 				(path "/dd07ab80-a59c-44f4-ac7d-849e21e1384e/3546f414-4018-45c7-a00a-bf02d214bf7f"
-					(reference "FB4")
+					(reference "FB3")
 					(unit 1)
 				)
@@
 		(dnp no)
 		(fields_autoplaced yes)
-		(property "Reference" "C121"
+		(property "Reference" "C101"
 			(at 45.72 148.5899 0)
 			(effects
@@
 			(project "mainboard4"
 				(path "/dd07ab80-a59c-44f4-ac7d-849e21e1384e/3546f414-4018-45c7-a00a-bf02d214bf7f"
-					(reference "C121")
+					(reference "C101")
 					(unit 1)
 				)
@@
 		(dnp no)
 		(fields_autoplaced yes)
-		(property "Reference" "C134"
+		(property "Reference" "C107"
 			(at 93.98 171.4499 0)
 			(effects
@@
 			(project "mainboard4"
 				(path "/dd07ab80-a59c-44f4-ac7d-849e21e1384e/3546f414-4018-45c7-a00a-bf02d214bf7f"
-					(reference "C134")
+					(reference "C107")
 					(unit 1)
 				)
@@
 		(dnp no)
 		(fields_autoplaced yes)
-		(property "Reference" "R61"
+		(property "Reference" "R57"
 			(at 140.97 68.58 90)
 			(effects
@@
 			(project "mainboard4"
 				(path "/dd07ab80-a59c-44f4-ac7d-849e21e1384e/3546f414-4018-45c7-a00a-bf02d214bf7f"
-					(reference "R61")
+					(reference "R57")
 					(unit 1)
 				)
@@
 		(dnp no)
 		(fields_autoplaced yes)
-		(property "Reference" "C100"
+		(property "Reference" "C87"
 			(at 107.95 35.5599 0)
 			(effects
@@
 			(project "mainboard4"
 				(path "/dd07ab80-a59c-44f4-ac7d-849e21e1384e/3546f414-4018-45c7-a00a-bf02d214bf7f"
-					(reference "C100")
+					(reference "C87")
 					(unit 1)
 				)
