File: CANFD.kicad_sch (KiCad schematic)
At the start: 9 parts, among them J2 Conn_01x04_Pin, U8 MCP2562-E-SN

Commit message: change cad data
Parts:
- renumbered C31 to C45, C37 to C52, D3 to D5, D4 to D6, J2 to J1, R21 to R30, R34 to R38, R35 to R41, U8 to U10
Connections:
- net VBUS renamed +12V
Changed lines of the file:
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@@
 		(on_board yes)
 		(dnp no)
-		(property "Reference" "D3"
+		(property "Reference" "D5"
 			(at 142.875 87.63 90)
 			(effects
@@
 			(project "mainboard4"
 				(path "/dd07ab80-a59c-44f4-ac7d-849e21e1384e/6416bab4-efd4-4cc0-95d7-68f4e661b691"
+					(reference "D5")
+					(unit 1)
+				)
+				(path "/dd07ab80-a59c-44f4-ac7d-849e21e1384e/edb81cb4-22a4-4ac0-9b4c-9e93cbd8a585"
 					(reference "D3")
-					(unit 1)
-				)
-				(path "/dd07ab80-a59c-44f4-ac7d-849e21e1384e/edb81cb4-22a4-4ac0-9b4c-9e93cbd8a585"
-					(reference "D5")
 					(unit 1)
 				)
@@
 		(on_board yes)
 		(dnp no)
-		(property "Reference" "U8"
+		(property "Reference" "U10"
 			(at 174.9141 83.185 0)
 			(effects
@@
 			(project ""
 				(path "/dd07ab80-a59c-44f4-ac7d-849e21e1384e/6416bab4-efd4-4cc0-95d7-68f4e661b691"
-					(reference "U8")
-					(unit 1)
-				)
-				(path "/dd07ab80-a59c-44f4-ac7d-849e21e1384e/edb81cb4-22a4-4ac0-9b4c-9e93cbd8a585"
-					(reference "U7")
+					(reference "U10")
+					(unit 1)
+				)
+				(path "/dd07ab80-a59c-44f4-ac7d-849e21e1384e/edb81cb4-22a4-4ac0-9b4c-9e93cbd8a585"
+					(reference "U9")
 					(unit 1)
 				)
@@
 		(dnp no)
 		(fields_autoplaced yes)
-		(property "Reference" "R34"
+		(property "Reference" "R38"
 			(at 147.955 81.915 0)
 			(effects
@@
 			(project "mainboard4"
 				(path "/dd07ab80-a59c-44f4-ac7d-849e21e1384e/6416bab4-efd4-4cc0-95d7-68f4e661b691"
-					(reference "R34")
-					(unit 1)
-				)
-				(path "/dd07ab80-a59c-44f4-ac7d-849e21e1384e/edb81cb4-22a4-4ac0-9b4c-9e93cbd8a585"
-					(reference "R31")
+					(reference "R38")
+					(unit 1)
+				)
+				(path "/dd07ab80-a59c-44f4-ac7d-849e21e1384e/edb81cb4-22a4-4ac0-9b4c-9e93cbd8a585"
+					(reference "R40")
 					(unit 1)
 				)
@@
 		(dnp no)
 		(fields_autoplaced yes)
-		(property "Reference" "J2"
+		(property "Reference" "J1"
 			(at 104.775 91.44 0)
 			(effects
@@
 			(project ""
 				(path "/dd07ab80-a59c-44f4-ac7d-849e21e1384e/6416bab4-efd4-4cc0-95d7-68f4e661b691"
+					(reference "J1")
+					(unit 1)
+				)
+				(path "/dd07ab80-a59c-44f4-ac7d-849e21e1384e/edb81cb4-22a4-4ac0-9b4c-9e93cbd8a585"
 					(reference "J2")
-					(unit 1)
-				)
-				(path "/dd07ab80-a59c-44f4-ac7d-849e21e1384e/edb81cb4-22a4-4ac0-9b4c-9e93cbd8a585"
-					(reference "J3")
 					(unit 1)
 				)
@@
 		(dnp no)
 		(fields_autoplaced yes)
-		(property "Reference" "R35"
+		(property "Reference" "R41"
 			(at 158.75 81.915 0)
 			(effects
@@
 			(project "mainboard4"
 				(path "/dd07ab80-a59c-44f4-ac7d-849e21e1384e/6416bab4-efd4-4cc0-95d7-68f4e661b691"
-					(reference "R35")
-					(unit 1)
-				)
-				(path "/dd07ab80-a59c-44f4-ac7d-849e21e1384e/edb81cb4-22a4-4ac0-9b4c-9e93cbd8a585"
-					(reference "R30")
-					(unit 1)
-				)
-			)
-		)
-	)
-	(symbol
-		(lib_id "power:VBUS")
-		(at 127 104.14 0)
-		(unit 1)
-		(exclude_from_sim no)
-		(in_bom yes)
-		(on_board yes)
-		(dnp no)
-		(fields_autoplaced yes)
-		(property "Reference" "#PWR0904"
-			(at 127 107.95 0)
-			(effects
-				(font
-					(size 1.27 1.27)
-				)
-				(hide yes)
-			)
-		)
-		(property "Value" "VBUS"
-			(at 127 99.06 0)
-			(effects
-				(font
-					(size 1.27 1.27)
-				)
-			)
-		)
-		(property "Footprint" ""
-			(at 127 104.14 0)
-			(effects
-				(font
-					(size 1.27 1.27)
-				)
-				(hide yes)
-			)
-		)
-		(property "Datasheet" ""
-			(at 127 104.14 0)
-			(effects
-				(font
-					(size 1.27 1.27)
-				)
-				(hide yes)
-			)
-		)
-		(property "Description" "Power symbol creates a global label with name \"VBUS\""
-			(at 127 104.14 0)
-			(effects
-				(font
-					(size 1.27 1.27)
-				)
-				(hide yes)
-			)
-		)
-		(pin "1"
-		)
-		(instances
-			(project ""
-				(path "/dd07ab80-a59c-44f4-ac7d-849e21e1384e/6416bab4-efd4-4cc0-95d7-68f4e661b691"
-					(reference "#PWR0704")
-					(unit 1)
-				)
-				(path "/dd07ab80-a59c-44f4-ac7d-849e21e1384e/edb81cb4-22a4-4ac0-9b4c-9e93cbd8a585"
-					(reference "#PWR0904")
+					(reference "R41")
+					(unit 1)
+				)
+				(path "/dd07ab80-a59c-44f4-ac7d-849e21e1384e/edb81cb4-22a4-4ac0-9b4c-9e93cbd8a585"
+					(reference "R39")
 					(unit 1)
 				)
@@
 		(dnp no)
 		(fields_autoplaced yes)
-		(property "Reference" "C31"
+		(property "Reference" "C45"
 			(at 203.2 92.7099 0)
 			(effects
@@
 			(project "mainboard4"
 				(path "/dd07ab80-a59c-44f4-ac7d-849e21e1384e/6416bab4-efd4-4cc0-95d7-68f4e661b691"
-					(reference "C31")
-					(unit 1)
-				)
-				(path "/dd07ab80-a59c-44f4-ac7d-849e21e1384e/edb81cb4-22a4-4ac0-9b4c-9e93cbd8a585"
-					(reference "C32")
+					(reference "C45")
+					(unit 1)
+				)
+				(path "/dd07ab80-a59c-44f4-ac7d-849e21e1384e/edb81cb4-22a4-4ac0-9b4c-9e93cbd8a585"
+					(reference "C48")
 					(unit 1)
 				)
@@
 		(on_board yes)
 		(dnp no)
-		(property "Reference" "R21"
+		(property "Reference" "R30"
 			(at 174.371 121.666 90)
 			(effects
@@
 			(project ""
 				(path "/dd07ab80-a59c-44f4-ac7d-849e21e1384e/6416bab4-efd4-4cc0-95d7-68f4e661b691"
-					(reference "R21")
-					(unit 1)
-				)
-				(path "/dd07ab80-a59c-44f4-ac7d-849e21e1384e/edb81cb4-22a4-4ac0-9b4c-9e93cbd8a585"
-					(reference "R20")
+					(reference "R30")
+					(unit 1)
+				)
+				(path "/dd07ab80-a59c-44f4-ac7d-849e21e1384e/edb81cb4-22a4-4ac0-9b4c-9e93cbd8a585"
+					(reference "R29")
 					(unit 1)
 				)
@@
 		(on_board yes)
 		(dnp no)
-		(property "Reference" "D4"
+		(property "Reference" "D6"
 			(at 153.035 87.63 90)
 			(effects
@@
 			(project "mainboard4"
 				(path "/dd07ab80-a59c-44f4-ac7d-849e21e1384e/6416bab4-efd4-4cc0-95d7-68f4e661b691"
+					(reference "D6")
+					(unit 1)
+				)
+				(path "/dd07ab80-a59c-44f4-ac7d-849e21e1384e/edb81cb4-22a4-4ac0-9b4c-9e93cbd8a585"
 					(reference "D4")
-					(unit 1)
-				)
-				(path "/dd07ab80-a59c-44f4-ac7d-849e21e1384e/edb81cb4-22a4-4ac0-9b4c-9e93cbd8a585"
-					(reference "D6")
 					(unit 1)
 				)
@@
 	)
 	(symbol
+		(lib_id "power:+12V")
+		(at 127 104.14 0)
+		(unit 1)
+		(exclude_from_sim no)
+		(in_bom yes)
+		(on_board yes)
+		(dnp no)
+		(fields_autoplaced yes)
+		(property "Reference" "#PWR01208"
+			(at 127 107.95 0)
+			(effects
+				(font
+					(size 1.27 1.27)
+				)
+				(hide yes)
+			)
+		)
+		(property "Value" "+12V"
+			(at 127 99.06 0)
+			(effects
+				(font
+					(size 1.27 1.27)
+				)
+			)
+		)
+		(property "Footprint" ""
+			(at 127 104.14 0)
+			(effects
+				(font
+					(size 1.27 1.27)
+				)
+				(hide yes)
+			)
+		)
+		(property "Datasheet" ""
+			(at 127 104.14 0)
+			(effects
+				(font
+					(size 1.27 1.27)
+				)
+				(hide yes)
+			)
+		)
+		(property "Description" "Power symbol creates a global label with name \"+12V\""
+			(at 127 104.14 0)
+			(effects
+				(font
+					(size 1.27 1.27)
+				)
+				(hide yes)
+			)
+		)
+		(pin "1"
+		)
+		(instances
+			(project "mainboard4"
+				(path "/dd07ab80-a59c-44f4-ac7d-849e21e1384e/6416bab4-efd4-4cc0-95d7-68f4e661b691"
+					(reference "#PWR01208")
+					(unit 1)
+				)
+				(path "/dd07ab80-a59c-44f4-ac7d-849e21e1384e/edb81cb4-22a4-4ac0-9b4c-9e93cbd8a585"
+					(reference "#PWR01301")
+					(unit 1)
+				)
+			)
+		)
+	)
+	(symbol
 		(lib_id "power:+5V")
 		(at 172.72 90.17 0)
@@
 		(dnp no)
 		(fields_autoplaced yes)
-		(property "Reference" "C37"
+		(property "Reference" "C52"
 			(at 151.13 107.9499 0)
 			(effects
@@
 			(project "mainboard4"
 				(path "/dd07ab80-a59c-44f4-ac7d-849e21e1384e/6416bab4-efd4-4cc0-95d7-68f4e661b691"
-					(reference "C37")
-					(unit 1)
-				)
-				(path "/dd07ab80-a59c-44f4-ac7d-849e21e1384e/edb81cb4-22a4-4ac0-9b4c-9e93cbd8a585"
-					(reference "C38")
-					(unit 1)
-				)
+					(reference "C52")
+					(unit 1)
+				)
+				(path "/dd07ab80-a59c-44f4-ac7d-849e21e1384e/edb81cb4-22a4-4ac0-9b4c-9e93cbd8a585"
+					(reference "C51")
+					(unit 1)
+				)

Commit message: remove efuse
Parts:
- renumbered C45 to C35, C52 to C42, R30 to R28, R38 to R37, R41 to R40, U10 to U11
Changed lines of the file:
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@@
 		(on_board yes)
 		(dnp no)
-		(property "Reference" "U10"
+		(property "Reference" "U11"
 			(at 174.9141 83.185 0)
 			(effects
@@
 			(project ""
 				(path "/dd07ab80-a59c-44f4-ac7d-849e21e1384e/6416bab4-efd4-4cc0-95d7-68f4e661b691"
+					(reference "U11")
+					(unit 1)
+				)
+				(path "/dd07ab80-a59c-44f4-ac7d-849e21e1384e/edb81cb4-22a4-4ac0-9b4c-9e93cbd8a585"
 					(reference "U10")
-					(unit 1)
-				)
-				(path "/dd07ab80-a59c-44f4-ac7d-849e21e1384e/edb81cb4-22a4-4ac0-9b4c-9e93cbd8a585"
-					(reference "U9")
 					(unit 1)
 				)
@@
 		(dnp no)
 		(fields_autoplaced yes)
-		(property "Reference" "R38"
+		(property "Reference" "R37"
 			(at 147.955 81.915 0)
 			(effects
@@
 			(project "mainboard4"
 				(path "/dd07ab80-a59c-44f4-ac7d-849e21e1384e/6416bab4-efd4-4cc0-95d7-68f4e661b691"
-					(reference "R38")
-					(unit 1)
-				)
-				(path "/dd07ab80-a59c-44f4-ac7d-849e21e1384e/edb81cb4-22a4-4ac0-9b4c-9e93cbd8a585"
-					(reference "R40")
+					(reference "R37")
+					(unit 1)
+				)
+				(path "/dd07ab80-a59c-44f4-ac7d-849e21e1384e/edb81cb4-22a4-4ac0-9b4c-9e93cbd8a585"
+					(reference "R39")
 					(unit 1)
 				)
@@
 		(dnp no)
 		(fields_autoplaced yes)
-		(property "Reference" "R41"
+		(property "Reference" "R40"
 			(at 158.75 81.915 0)
 			(effects
@@
 			(project "mainboard4"
 				(path "/dd07ab80-a59c-44f4-ac7d-849e21e1384e/6416bab4-efd4-4cc0-95d7-68f4e661b691"
-					(reference "R41")
-					(unit 1)
-				)
-				(path "/dd07ab80-a59c-44f4-ac7d-849e21e1384e/edb81cb4-22a4-4ac0-9b4c-9e93cbd8a585"
-					(reference "R39")
+					(reference "R40")
+					(unit 1)
+				)
+				(path "/dd07ab80-a59c-44f4-ac7d-849e21e1384e/edb81cb4-22a4-4ac0-9b4c-9e93cbd8a585"
+					(reference "R38")
 					(unit 1)
 				)
@@
 		(dnp no)
 		(fields_autoplaced yes)
-		(property "Reference" "C45"
+		(property "Reference" "C35"
 			(at 203.2 92.7099 0)
 			(effects
@@
 			(project "mainboard4"
 				(path "/dd07ab80-a59c-44f4-ac7d-849e21e1384e/6416bab4-efd4-4cc0-95d7-68f4e661b691"
-					(reference "C45")
-					(unit 1)
-				)
-				(path "/dd07ab80-a59c-44f4-ac7d-849e21e1384e/edb81cb4-22a4-4ac0-9b4c-9e93cbd8a585"
-					(reference "C48")
+					(reference "C35")
+					(unit 1)
+				)
+				(path "/dd07ab80-a59c-44f4-ac7d-849e21e1384e/edb81cb4-22a4-4ac0-9b4c-9e93cbd8a585"
+					(reference "C38")
 					(unit 1)
 				)
@@
 		(on_board yes)
 		(dnp no)
-		(property "Reference" "R30"
+		(property "Reference" "R28"
 			(at 174.371 121.666 90)
 			(effects
@@
 			(project ""
 				(path "/dd07ab80-a59c-44f4-ac7d-849e21e1384e/6416bab4-efd4-4cc0-95d7-68f4e661b691"
-					(reference "R30")
-					(unit 1)
-				)
-				(path "/dd07ab80-a59c-44f4-ac7d-849e21e1384e/edb81cb4-22a4-4ac0-9b4c-9e93cbd8a585"
-					(reference "R29")
+					(reference "R28")
+					(unit 1)
+				)
+				(path "/dd07ab80-a59c-44f4-ac7d-849e21e1384e/edb81cb4-22a4-4ac0-9b4c-9e93cbd8a585"
+					(reference "R27")
 					(unit 1)
 				)
@@
 		(dnp no)
 		(fields_autoplaced yes)
-		(property "Reference" "C52"
+		(property "Reference" "C42"
 			(at 151.13 107.9499 0)
 			(effects
@@
 			(project "mainboard4"
 				(path "/dd07ab80-a59c-44f4-ac7d-849e21e1384e/6416bab4-efd4-4cc0-95d7-68f4e661b691"
-					(reference "C52")
-					(unit 1)
-				)
-				(path "/dd07ab80-a59c-44f4-ac7d-849e21e1384e/edb81cb4-22a4-4ac0-9b4c-9e93cbd8a585"
-					(reference "C51")
-					(unit 1)
-				)
+					(reference "C42")
+					(unit 1)
+				)
+				(path "/dd07ab80-a59c-44f4-ac7d-849e21e1384e/edb81cb4-22a4-4ac0-9b4c-9e93cbd8a585"
+					(reference "C41")
+					(unit 1)
+				)

Commit message: add sata capacitor
Parts:
- renumbered C35 to C43, C42 to C50, D6 to D5, D5 to D6, J1 to J2, R37 to R38, R40 to R39, U11 to U10
Changed lines of the file:
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@@
 	(label "CANH"
 		(at 190.5 99.06 180)
+		(fields_autoplaced yes)
 		(effects
 			(font
@@
 	(label "CANH"
 		(at 167.64 127 180)
+		(fields_autoplaced yes)
 		(effects
 			(font
@@
 	(label "CANH"
 		(at 119.38 101.6 0)
+		(fields_autoplaced yes)
 		(effects
 			(font
@@
 	(label "CANL"
 		(at 190.5 104.14 180)
+		(fields_autoplaced yes)
 		(effects
 			(font
@@
 	(label "CANL"
 		(at 175.26 127 0)
+		(fields_autoplaced yes)
 		(effects
 			(font
@@
 	(label "CANL"
 		(at 119.38 99.06 0)
+		(fields_autoplaced yes)
 		(effects
 			(font
@@
 		(shape output)
 		(at 142.24 99.06 180)
+		(fields_autoplaced yes)
 		(effects
 			(font
@@
 		(shape input)
 		(at 142.24 96.52 180)
+		(fields_autoplaced yes)
 		(effects
 			(font
@@
 		(on_board yes)
 		(dnp no)
-		(property "Reference" "D5"
+		(property "Reference" "D6"
 			(at 142.875 87.63 90)
 			(effects
@@
 			(project "mainboard4"
 				(path "/dd07ab80-a59c-44f4-ac7d-849e21e1384e/6416bab4-efd4-4cc0-95d7-68f4e661b691"
-					(reference "D5")
+					(reference "D6")
 					(unit 1)
 				)
@@
 		(on_board yes)
 		(dnp no)
-		(property "Reference" "U11"
+		(property "Reference" "U10"
 			(at 174.9141 83.185 0)
 			(effects
@@
 			(project ""
 				(path "/dd07ab80-a59c-44f4-ac7d-849e21e1384e/6416bab4-efd4-4cc0-95d7-68f4e661b691"
+					(reference "U10")
+					(unit 1)
+				)
+				(path "/dd07ab80-a59c-44f4-ac7d-849e21e1384e/edb81cb4-22a4-4ac0-9b4c-9e93cbd8a585"
 					(reference "U11")
-					(unit 1)
-				)
-				(path "/dd07ab80-a59c-44f4-ac7d-849e21e1384e/edb81cb4-22a4-4ac0-9b4c-9e93cbd8a585"
-					(reference "U10")
 					(unit 1)
 				)
@@
 		(dnp no)
 		(fields_autoplaced yes)
-		(property "Reference" "R37"
+		(property "Reference" "R38"
 			(at 147.955 81.915 0)
 			(effects
@@
 			(project "mainboard4"
 				(path "/dd07ab80-a59c-44f4-ac7d-849e21e1384e/6416bab4-efd4-4cc0-95d7-68f4e661b691"
-					(reference "R37")
-					(unit 1)
-				)
-				(path "/dd07ab80-a59c-44f4-ac7d-849e21e1384e/edb81cb4-22a4-4ac0-9b4c-9e93cbd8a585"
-					(reference "R39")
+					(reference "R38")
+					(unit 1)
+				)
+				(path "/dd07ab80-a59c-44f4-ac7d-849e21e1384e/edb81cb4-22a4-4ac0-9b4c-9e93cbd8a585"
+					(reference "R40")
 					(unit 1)
 				)
@@
 		(dnp no)
 		(fields_autoplaced yes)
-		(property "Reference" "J1"
+		(property "Reference" "J2"
 			(at 104.775 91.44 0)
 			(effects
@@
 			(project ""
 				(path "/dd07ab80-a59c-44f4-ac7d-849e21e1384e/6416bab4-efd4-4cc0-95d7-68f4e661b691"
+					(reference "J2")
+					(unit 1)
+				)
+				(path "/dd07ab80-a59c-44f4-ac7d-849e21e1384e/edb81cb4-22a4-4ac0-9b4c-9e93cbd8a585"
 					(reference "J1")
-					(unit 1)
-				)
-				(path "/dd07ab80-a59c-44f4-ac7d-849e21e1384e/edb81cb4-22a4-4ac0-9b4c-9e93cbd8a585"
-					(reference "J2")
 					(unit 1)
 				)
@@
 		(dnp no)
 		(fields_autoplaced yes)
-		(property "Reference" "R40"
+		(property "Reference" "R39"
 			(at 158.75 81.915 0)
 			(effects
@@
 			(project "mainboard4"
 				(path "/dd07ab80-a59c-44f4-ac7d-849e21e1384e/6416bab4-efd4-4cc0-95d7-68f4e661b691"
-					(reference "R40")
-					(unit 1)
-				)
-				(path "/dd07ab80-a59c-44f4-ac7d-849e21e1384e/edb81cb4-22a4-4ac0-9b4c-9e93cbd8a585"
-					(reference "R38")
+					(reference "R39")
+					(unit 1)
+				)
+				(path "/dd07ab80-a59c-44f4-ac7d-849e21e1384e/edb81cb4-22a4-4ac0-9b4c-9e93cbd8a585"
+					(reference "R41")
 					(unit 1)
 				)
@@
 		(dnp no)
 		(fields_autoplaced yes)
-		(property "Reference" "C35"
+		(property "Reference" "C43"
 			(at 203.2 92.7099 0)
 			(effects
@@
 			(project "mainboard4"
 				(path "/dd07ab80-a59c-44f4-ac7d-849e21e1384e/6416bab4-efd4-4cc0-95d7-68f4e661b691"
-					(reference "C35")
-					(unit 1)
-				)
-				(path "/dd07ab80-a59c-44f4-ac7d-849e21e1384e/edb81cb4-22a4-4ac0-9b4c-9e93cbd8a585"
-					(reference "C38")
+					(reference "C43")
+					(unit 1)
+				)
+				(path "/dd07ab80-a59c-44f4-ac7d-849e21e1384e/edb81cb4-22a4-4ac0-9b4c-9e93cbd8a585"
+					(reference "C44")
 					(unit 1)
 				)
@@
 		(on_board yes)
 		(dnp no)
-		(property "Reference" "D6"
+		(property "Reference" "D5"
 			(at 153.035 87.63 90)
 			(effects
@@
 			(project "mainboard4"
 				(path "/dd07ab80-a59c-44f4-ac7d-849e21e1384e/6416bab4-efd4-4cc0-95d7-68f4e661b691"
-					(reference "D6")
+					(reference "D5")
 					(unit 1)
 				)
@@
 		(dnp no)
 		(fields_autoplaced yes)
-		(property "Reference" "C42"
+		(property "Reference" "C50"
 			(at 151.13 107.9499 0)
 			(effects
@@
 			(project "mainboard4"
 				(path "/dd07ab80-a59c-44f4-ac7d-849e21e1384e/6416bab4-efd4-4cc0-95d7-68f4e661b691"
-					(reference "C42")
-					(unit 1)
-				)
-				(path "/dd07ab80-a59c-44f4-ac7d-849e21e1384e/edb81cb4-22a4-4ac0-9b4c-9e93cbd8a585"
-					(reference "C41")
-					(unit 1)
-				)
+					(reference "C50")
+					(unit 1)
+				)
+				(path "/dd07ab80-a59c-44f4-ac7d-849e21e1384e/edb81cb4-22a4-4ac0-9b4c-9e93cbd8a585"
+					(reference "C49")
+					(unit 1)
+				)

Commit message: add logp
Parts:
- renumbered R28 to R25, R38 to R35, R39 to R36
Changed lines of the file:
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@@
 	(label "CANH"
 		(at 190.5 99.06 180)
-		(fields_autoplaced yes)
 		(effects
 			(font
@@
 	(label "CANH"
 		(at 167.64 127 180)
-		(fields_autoplaced yes)
 		(effects
 			(font
@@
 	(label "CANH"
 		(at 119.38 101.6 0)
-		(fields_autoplaced yes)
 		(effects
 			(font
@@
 	(label "CANL"
 		(at 190.5 104.14 180)
-		(fields_autoplaced yes)
 		(effects
 			(font
@@
 	(label "CANL"
 		(at 175.26 127 0)
-		(fields_autoplaced yes)
 		(effects
 			(font
@@
 	(label "CANL"
 		(at 119.38 99.06 0)
-		(fields_autoplaced yes)
 		(effects
 			(font
@@
 		(shape output)
 		(at 142.24 99.06 180)
-		(fields_autoplaced yes)
 		(effects
 			(font
@@
 		(shape input)
 		(at 142.24 96.52 180)
-		(fields_autoplaced yes)
 		(effects
 			(font
@@
 		(dnp no)
 		(fields_autoplaced yes)
-		(property "Reference" "R38"
+		(property "Reference" "R35"
 			(at 147.955 81.915 0)
 			(effects
@@
 			(project "mainboard4"
 				(path "/dd07ab80-a59c-44f4-ac7d-849e21e1384e/6416bab4-efd4-4cc0-95d7-68f4e661b691"
-					(reference "R38")
-					(unit 1)
-				)
-				(path "/dd07ab80-a59c-44f4-ac7d-849e21e1384e/edb81cb4-22a4-4ac0-9b4c-9e93cbd8a585"
-					(reference "R40")
+					(reference "R35")
+					(unit 1)
+				)
+				(path "/dd07ab80-a59c-44f4-ac7d-849e21e1384e/edb81cb4-22a4-4ac0-9b4c-9e93cbd8a585"
+					(reference "R37")
 					(unit 1)
 				)
@@
 		(dnp no)
 		(fields_autoplaced yes)
-		(property "Reference" "R39"
+		(property "Reference" "R36"
 			(at 158.75 81.915 0)
 			(effects
@@
 			(project "mainboard4"
 				(path "/dd07ab80-a59c-44f4-ac7d-849e21e1384e/6416bab4-efd4-4cc0-95d7-68f4e661b691"
-					(reference "R39")
-					(unit 1)
-				)
-				(path "/dd07ab80-a59c-44f4-ac7d-849e21e1384e/edb81cb4-22a4-4ac0-9b4c-9e93cbd8a585"
-					(reference "R41")
+					(reference "R36")
+					(unit 1)
+				)
+				(path "/dd07ab80-a59c-44f4-ac7d-849e21e1384e/edb81cb4-22a4-4ac0-9b4c-9e93cbd8a585"
+					(reference "R38")
 					(unit 1)
 				)
@@
 		(on_board yes)
 		(dnp no)
-		(property "Reference" "R28"
+		(property "Reference" "R25"
 			(at 174.371 121.666 90)
 			(effects
@@
 			(project ""
 				(path "/dd07ab80-a59c-44f4-ac7d-849e21e1384e/6416bab4-efd4-4cc0-95d7-68f4e661b691"
-					(reference "R28")
-					(unit 1)
-				)
-				(path "/dd07ab80-a59c-44f4-ac7d-849e21e1384e/edb81cb4-22a4-4ac0-9b4c-9e93cbd8a585"
-					(reference "R27")
-					(unit 1)
-				)
+					(reference "R25")
+					(unit 1)
+				)
+				(path "/dd07ab80-a59c-44f4-ac7d-849e21e1384e/edb81cb4-22a4-4ac0-9b4c-9e93cbd8a585"
+					(reference "R24")
+					(unit 1)
+				)

Commit message: データをアップロード
Parts:
- removed D5: LED, LED_SMD:LED_0603_1608Metric_Pad1.05x0.95mm_HandSolder, symbol Device:LED
- removed J2: Conn_01x04_Pin, CM5IO:pocketheader4, symbol Connector:Conn_01x04_Pin
- removed R35, R36: 1k, Resistor_SMD:R_0603_1608Metric_Pad0.98x0.95mm_HandSolder, symbol Device:R
- added D8: LED, LED_SMD:LED_0603_1608Metric_Pad1.05x0.95mm_HandSolder, symbol Device:LED
- added J3: Conn_01x04_Pin, CM5IO:pocketheader4, symbol Connector:Conn_01x04_Pin
- added R3, R5: 1k, Resistor_SMD:R_0603_1608Metric_Pad0.98x0.95mm_HandSolder, symbol Device:R
- C47: renamed from C50; footprint Capacitor_SMD:C_0402_1005Metric_Pad0.74x0.62mm_HandSolder -> Capacitor_SMD:C_0603_1608Metric_Pad1.08x0.95mm_HandSolder
- C54: renamed from C43; footprint Capacitor_SMD:C_0402_1005Metric_Pad0.74x0.62mm_HandSolder -> Capacitor_SMD:C_0603_1608Metric_Pad1.08x0.95mm_HandSolder
- renumbered R25 to R31, U10 to U11
Connections:
- net +12V: now also J3.1 (Pin_1)
- net +3.3V: now also R3.1, R5.1
- net CANRX: now also D8.1 (K)
- net GND: now also J3.4 (Pin_4)
- net at D6.2 (A): now also R3.2
- net CANH renamed CANP
- net CANP: now also J3.2 (Pin_2)
- net CANL renamed CANN
- net CANN: now also J3.3 (Pin_3)
- new net: D8.2 (A), R5.2
Other:
- moved on the sheet: C47, C54, R31, U11
