File: MCU.kicad_sch (KiCad schematic)
At the start: 18 parts, among them J6 Conn_02x07_Odd_Even, SW3 SW_Push, U12 STM32H723VGT6, Y2 16Mhz

Commit message: データをアップロード
Parts:
- C9: renamed from C16; footprint Capacitor_SMD:C_0603_1608Metric_Pad1.08x0.95mm_HandSolder -> Capacitor_SMD:C_0402_1005Metric_Pad0.74x0.62mm_HandSolder
- J1: renamed from J6; footprint CM5IO:connector -> CM5symbol:connector
- R16: renamed from R27; value 12kΩ -> 10kΩ; footprint Resistor_SMD:R_0603_1608Metric_Pad0.98x0.95mm_HandSolder -> Resistor_SMD:R_0402_1005Metric_Pad0.72x0.64mm_HandSolder
- renumbered C48 to C1, C55 to C11, C51 to C12, C63 to C15, C58 to C16, C47 to C2, C45 to C3, C46 to C4, C52 to C6, C62 to C8, D7 to D3, SW3 to SW2, U12 to U2, Y2 to Y1
Connections:
- net USART2_RX is gone; now on net UART_RX: J1.13 (Pin_13)
- net USART2_TX is gone; now on net UART_TX: J1.14 (Pin_14)
- net CAN1RX: now also U2.59 (PD12); no longer U2.81 (PD0)
- net CAN1TX: now also U2.60 (PD13); no longer U2.82 (PD1)
- net CAN2RX: now also U2.82 (PD1); no longer U2.91 (PB5)
- net CAN2TX: now also U2.81 (PD0); no longer U2.92 (PB6)
- net CS: now also U2.41 (PE11); no longer U2.3 (PE4)
- net INT: now also U2.45 (PE15); no longer U2.97 (PE0)
- net LED: now also U2.39 (PE9); no longer U2.67 (PA8)
- net MISO: now also U2.43 (PE13); no longer U2.4 (PE5)
- net MOSI: now also U2.44 (PE14); no longer U2.5 (PE6)
- net RST: now also U2.40 (PE10); no longer U2.98 (PE1)
- net SCLK: now also U2.42 (PE12); no longer U2.1 (PE2)
- net UART_RX: now reaches U2.37 (PE7)
- net UART_TX: now reaches U2.38 (PE8)
- net CRS_DV renamed CRSDV
- net ETH_REF_CLK renamed REFCLK
- net GNDDETECT: no longer names the net of J1.11 (Pin_11)
- net NRST renamed ~{RESET}
- net TX_EN renamed TXEN
- net T_SWCLK renamed SWCLK
- net T_SWDIO renamed SWDIO
- net T_SWO renamed SWO
- net USB_DN renamed MCU.DN
- net USB_DP renamed MCU.DP
Other:
- moved on the sheet: C1, C11, C12, C16, C3, C4, C6, C8, C9, D3, FB1, J1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
