File: NVME.kicad_sch (KiCad schematic)
At the start: 11 parts, among them J7 Bus_M.2_Socket_E, U12 ASEK-32.768KHZ-L-R-T

Commit message: データをアップロード
Parts:
- removed C25, C26, C29: 0.1uF, Capacitor_SMD:C_0603_1608Metric, symbol Device:C
- removed C28: 0.01uF, Capacitor_SMD:C_0603_1608Metric, symbol Device:C
- removed C60: 100n, Capacitor_SMD:C_0402_1005Metric_Pad0.74x0.62mm_HandSolder, symbol Device:C
- removed D11: LED Green, LED_SMD:LED_0603_1608Metric_Pad1.05x0.95mm_HandSolder, symbol Device:LED
- removed J7: Bus_M.2_Socket_E, CM5IO:M.2 E Key socket, symbol Connector:Bus_M.2_Socket_E
- removed R36: 1k, Resistor_SMD:R_0603_1608Metric_Pad0.98x0.95mm_HandSolder, symbol Device:R
- removed R37: 1k, Resistor_SMD:R_0402_1005Metric_Pad0.72x0.64mm_HandSolder, symbol Device:R
- removed R38: 100k, Resistor_SMD:R_0402_1005Metric_Pad0.72x0.64mm_HandSolder, symbol Device:R
- removed U12: ASEK-32.768KHZ-L-R-T, Crystal:Crystal_SMD_3225-4Pin_3.2x2.5mm, symbol CM5IO:ASEK-32.768KHZ-L-R-T
- added C13, C5, C7: 0.1uF, Capacitor_SMD:C_0603_1608Metric, symbol Device:C
- added C14: 0.01uF, Capacitor_SMD:C_0603_1608Metric, symbol Device:C
- added C17: 100n, Capacitor_SMD:C_0402_1005Metric_Pad0.74x0.62mm_HandSolder, symbol Device:C
- added D10: LED Green, LED_SMD:LED_0603_1608Metric_Pad1.05x0.95mm_HandSolder, symbol Device:LED
- added J2: Bus_M.2_Socket_M, CM5symbol:M.2 M Key socket, symbol Connector:Bus_M.2_Socket_M
- added R35: 1k, Resistor_SMD:R_0603_1608Metric_Pad0.98x0.95mm_HandSolder, symbol Device:R
- added U4: ASEK-32.768KHZ-L-R-T, Crystal:Crystal_SMD_3225-4Pin_3.2x2.5mm, symbol CM5IO:ASEK-32.768KHZ-L-R-T
Connections:
- net +3.3V: now also C13.1, C14.1, C17.1, C5.1, C7.1, D10.2 (A), J2.12 (3.3V), J2.14 (3.3V), J2.16 (3.3V), J2.18 (3.3V), J2.2 (3.3V), J2.4 (3.3V), J2.70 (3.3V), J2.72 (3.3V), J2.74 (3.3V), U4.1 (EN), U4.4 (VDD)
- net GND: now also C13.2, C14.2, C17.2, C5.2, C7.2, J2.1 (GND), J2.15 (GND), J2.21 (GND), J2.27 (GND), J2.3 (GND), J2.33 (GND), J2.39 (GND), J2.45 (GND), J2.51 (GND), J2.57 (GND), J2.71 (GND), J2.73 (GND), J2.75 (GND), J2.9 (GND), U4.2 (GND)
- net nRST: now also J2.50 (~{PERST})
- new net: J2.10 (DAS/~{DSS}/~{LED1}), R35.2
- new net: J2.68 (SUSCLK), U4.3 (Out)
- new net: D10.1 (K), R35.1
- new net NVME.CLKN: J2.55 (REFCLKp)
- new net NVME.CLKP: J2.53 (REFCLKn)
- new net NVME.RXN: J2.43 (PERp0/SATA-B-)
- new net NVME.RXP: J2.41 (PERn0/SATA-B+)
- new net NVME.TXN: J2.47 (PETn0/SATA-A-)
- new net NVME.TXP: J2.49 (PETp0/SATA-A+)
- no-connect marks 0 -> 16
Other:
- note removed: "Activity LED"
- company: Copyright © 2024 Raspberry Pi Ltd. -> (none)
- title: Compute Module 5 IO Board - M2 Socket -> (none)
