File: mainboard4.kicad_sch (KiCad schematic)
At the start: 9 parts, among them J12 USB3_A, J13 USB_C_Receptacle_USB2.0_16P, J8 Barrel_Jack

Commit message: end route
Parts:
- renumbered C109 to C79, C110 to C80, J8 to J9
Changed lines of the file:
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@@
 		(on_board yes)
 		(dnp no)
-		(property "Reference" "C110"
+		(property "Reference" "C80"
 			(at 143.51 47.752 0)
 			(effects
@@
 			(project "mainboard4"
 				(path "/dd07ab80-a59c-44f4-ac7d-849e21e1384e"
-					(reference "C110")
+					(reference "C80")
 					(unit 1)
 				)
@@
 		(on_board yes)
 		(dnp no)
-		(property "Reference" "J8"
+		(property "Reference" "J9"
 			(at 24.3078 172.085 0)
 			(effects
@@
 			(project "mainboard4"
 				(path "/dd07ab80-a59c-44f4-ac7d-849e21e1384e"
-					(reference "J8")
+					(reference "J9")
 					(unit 1)
 				)
@@
 		(on_board yes)
 		(dnp no)
-		(property "Reference" "C109"
+		(property "Reference" "C79"
 			(at 130.81 52.07 0)
 			(effects
@@
 			(project "mainboard4"
 				(path "/dd07ab80-a59c-44f4-ac7d-849e21e1384e"
-					(reference "C109")
-					(unit 1)
-				)
+					(reference "C79")
+					(unit 1)
+				)

Commit message: データをアップロード
Parts:
- removed C64, C65, C66, C67, C79, C80: 0.1uF, Capacitor_SMD:C_0402_1005Metric_Pad0.74x0.62mm_HandSolder, symbol Device:C
- removed J12: USB3_A, CM5IO:MTCONN_UBAF30-D2011, symbol CM5IO:USB3_A
Other:
- sheet CM5_GPIO renamed CM5_INTERFACE
- sheet CM5_HighSpeed renamed CM5
- sheet CM5_PCIe renamed WiFi_PCIe
- removed sheet IMU
- removed sheet USB2Ethernet
- removed sheet USB2SATA
- added sheet NIC (NIC.kicad_sch)
- added sheet NVME (NVME.kicad_sch)
- added sheet PCIe_SW (PCIe_SW.kicad_sch)
- added sheet USB (USB.kicad_sch)
- sheet CM5: file CM5_HighSpeed.kicad_sch -> CM5.kicad_sch
- sheet CM5 ports: added HOST{PCIe}, LED_nACT, PCIe_nRST, POWER_SW, USB0{USB3.0}, USB1{USB3.0}, USB2{USB2.0}, nPWR_LED, {CONFIG}, {Ethernet}, {FAN}, {GPDI}, {GPIO}, {SDMMC}, {TouchDisplay}; removed PCIE_CLK_N, PCIE_CLK_P, PCIE_PWR_EN, PCIE_RX_N, PCIE_RX_P, PCIE_TX_N, PCIE_TX_P, PCIE_nCLKREQ, PCIE_nRST, PCIE_nWAKE, USB2_N, USB2_P, USB3-0-D_N, USB3-0-D_P, USB3-0-RX_N, USB3-0-RX_P, USB3-0-TX_N, USB3-0-TX_P, USB3-1-D_N, USB3-1-D_P, USB3-1-RX_N, USB3-1-RX_P, USB3-1-TX_N, USB3-1-TX_P
- sheet CM5_INTERFACE ports: added LED_nACT, POWER_SW, nPWR_LED, {CONFIG}, {FAN}, {GPDI}, {GPIO}, {SDMMC}, {TouchDisplay}; removed RESET
- sheet Ethernet PHY ports: added {Ethernet}, {RMII}; removed CRSDV, MDC, MDIO, REFCLK, RXD0, RXD1, RXN, RXP, TXD0, TXD1, TXEN, TXN, TXP
- sheet MCU ports: added MCU{USB2.0}, {RMII}; removed CRS_DV, CS, ETH_REF_CLK, INT, MDC, MDIO, MISO, MOSI, RST, RXD0, RXD1, SCLK, TXD0, TXD1, TX_EN, USB_DN, USB_DP
- sheet Power ports: added none; removed 3.3V, 5V, 5V_VBUS, VBUS_EN
- sheet WiFi_PCIe ports: added WiFi{PCIe}, WiFi{USB2.0}, nRST; removed PCIE_CLK_N, PCIE_CLK_P, PCIE_PWR_EN, PCIE_RX_N, PCIE_RX_P, PCIE_TX_N, PCIE_TX_P, PCIE_nCLKREQ, PCIE_nRST, PCIE_nWAKE, USB_D+, USB_D-
- note removed: "USB 3 Pairs P/N swapped to help routing"
- moved on the sheet: J13, J9
